File: KiCad/Motion controller MiYR interface/Motion controller MiYR interface.kicad_pcb (KiCad board)
At the start: 4 copper layers, 86 x 198 mm, 101 parts, among them CN1 Conn_02x40_Odd_Even, CN2 Conn_02x40_Odd_Even, J1 10061913-111PLF, J2 10061913-111PLF, J3 10061913-111PLF, J4 10061913-111PLF, J5 Conn_01x02_Pin, U1 AP63201WU, U10 D1213A-04S-7, U11 D1213A-04S-7, U12 D1213A-04S-7, U13 D1213A-04S-7, U14 D1213A-04S-7, U15 D1213A-04S-7, U16 D1213A-04S-7, U17 D1213A-04S-7, U18 D1213A-04S-7, U19 D1213A-04S-7, U2 AOZ1360AIL, U20 D1213A-04S-7, U21 D1213A-04S-7, U22 D1213A-04S-7, U23 AOZ1360AIL, U24 AP63201WU, U25 AOZ1360AIL, U26 AP63201WU, U3 D1213A-04S-7, U30 D1213A-04S-7, U31 D1213A-04S-7, U32 D1213A-04S-7, U33 D1213A-04S-7, U4 D1213A-04S-7, U5 D1213A-04S-7, U6 D1213A-04S-7, U7 D1213A-04S-7, U8 D1213A-04S-7, U9 D1213A-04S-7

Commit message: update
Parts:
- removed C20, C31: 100pf, Capacitor_SMD:C_0603_1608Metric
- removed C21, C22, C29, C32, C33: 10uf, Capacitor_SMD:C_1206_3216Metric
- removed C30: .1uf, Capacitor_SMD:C_0603_1608Metric
- removed L3: 6.8uH, Inductor_SMD:L_Taiyo-Yuden_MD-5050
- removed R15: 100k, Resistor_SMD:R_0603_1608Metric
- removed the REF** at (211.0, 157.0)
- removed the REF** at (211.0, 115.0)
- removed the REF** at (132.5, 55.0)
- removed the REF** at (132.5, 91.0)
- removed the REF** at (202.0, 236.0)
- removed the REF** at (144.0, 238.0)
- removed the REF** at (211.0, 74.0)
- removed the REF** at (211.0, 245.0)
- removed the REF** at (211.0, 201.0)
- removed the REF** at (132.5, 245.0)
- removed the REF** at (200.0, 238.0)
- removed the REF** at (132.5, 201.0)
- removed the REF** at (140.2, 237.2)
- removed the REF** at (132.5, 157.0)
- removed U23: AOZ1360AIL, footprints:AOZ1360AIL_AOS
- removed U24, U26: AP63201WU, Package_TO_SOT_SMD:TSOT-23-6
- added C36: 75pf, Capacitor_SMD:C_0402_1005Metric, F.Cu at (152.8, 68.6)
- added C37: 22uf, Capacitor_SMD:C_1206_3216Metric, F.Cu at (155.6, 69.6)
- added C38: 22uf, Capacitor_SMD:C_1206_3216Metric, F.Cu at (160.3, 69.6)
- added C48: 10uf, Capacitor_SMD:C_1206_3216Metric, F.Cu at (184.9, 95.6)
- added C50: 10uf, Capacitor_SMD:C_1206_3216Metric, F.Cu at (184.4, 142.6)
- added C70: 10uf, Capacitor_SMD:C_1206_3216Metric, F.Cu at (184.6, 189.5)
- added C72: 10uf, Capacitor_SMD:C_1206_3216Metric, F.Cu at (184.7, 236.5)
- added C74: 10uf, Capacitor_SMD:C_1206_3216Metric, F.Cu at (202.6, 238.8)
- added D10: LED, LED_SMD:LED_0603_1608Metric, B.Cu at (183.6, 84.8)
- added D11: LED, LED_SMD:LED_0603_1608Metric, B.Cu at (183.5, 131.6)
- added D12: LED, LED_SMD:LED_0603_1608Metric, B.Cu at (183.6, 178.5)
- added D13: LED, LED_SMD:LED_0603_1608Metric, B.Cu at (183.4, 225.8)
- added D14: LED, LED_SMD:LED_0603_1608Metric, B.Cu at (170.5, 60.0)
- added D15: LED, LED_SMD:LED_0603_1608Metric, B.Cu at (158.7, 73.7)
- added D16: LED, LED_SMD:LED_0603_1608Metric, B.Cu at (146.2, 73.7)
- added D18: SS34, Diode_SMD:D_SMA, F.Cu at (198.3, 65.9)
- added D19: SS34, Diode_SMD:D_SMA, F.Cu at (184.6, 91.5)
- added D2: LED, LED_SMD:LED_0603_1608Metric, B.Cu at (170.5, 73.7)
- added D20: SS34, Diode_SMD:D_SMA, F.Cu at (184.5, 138.6)
- added D21: SS34, Diode_SMD:D_SMA, F.Cu at (184.6, 185.6)
- added D22: SS34, Diode_SMD:D_SMA, F.Cu at (184.8, 232.6)
- added D3: LED, LED_SMD:LED_0603_1608Metric, B.Cu at (183.4, 73.7)
- added F2: 3A, Fuse:Fuse_2920_7451Metric, F.Cu at (188.0, 86.0)
- added F3: 3A, Fuse:Fuse_2920_7451Metric, F.Cu at (188.0, 132.7)
- added F4: 3A, Fuse:Fuse_2920_7451Metric, F.Cu at (188.0, 179.6)
- added F5: 3A, Fuse:Fuse_2920_7451Metric, F.Cu at (188.0, 226.9)
- added H1: MountingHole, MountingHole:MountingHole_3.2mm_M3, F.Cu at (132.5, 55.0)
- added H10: MountingHole, MountingHole:MountingHole_3.2mm_M3, F.Cu at (211.0, 245.0)
- added H2: MountingHole, MountingHole:MountingHole_3.2mm_M3, F.Cu at (132.5, 91.0)
- added H3: MountingHole, MountingHole:MountingHole_3.2mm_M3, F.Cu at (132.5, 157.0)
- added H4: MountingHole, MountingHole:MountingHole_3.2mm_M3, F.Cu at (132.5, 201.0)
- added H5: MountingHole, MountingHole:MountingHole_3.2mm_M3, F.Cu at (132.5, 245.0)
- added H6: MountingHole, MountingHole:MountingHole_3.2mm_M3, F.Cu at (211.0, 74.0)
- added H7: MountingHole, MountingHole:MountingHole_3.2mm_M3, F.Cu at (211.0, 115.0)
- added H8: MountingHole, MountingHole:MountingHole_3.2mm_M3, F.Cu at (211.0, 157.0)
- added H9: MountingHole, MountingHole:MountingHole_3.2mm_M3, F.Cu at (211.0, 201.0)
- added L4: 15uH, footprints:CY54_INDUCTOR, F.Cu at (160.2, 65.2)
- added M1: Fan, Connector_PinHeader_2.54mm:PinHeader_1x02_P2.54mm_Vertical, B.Cu at (203.8, 242.2)
- added M2: Fan, Connector_PinHeader_2.54mm:PinHeader_1x02_P2.54mm_Vertical, B.Cu at (192.3, 55.9)
- added R10: 100k, Resistor_SMD:R_0402_1005Metric, F.Cu at (154.1, 61.5)
- added R11: 100k, Resistor_SMD:R_0402_1005Metric, F.Cu at (151.8, 68.6)
- added R12: 13.3k, Resistor_SMD:R_0402_1005Metric, F.Cu at (154.1, 62.5)
- added R17: 1k, Resistor_SMD:R_0402_1005Metric, F.Cu at (174.4, 72.6)
- added R18: 1k, Resistor_SMD:R_0402_1005Metric, F.Cu at (187.9, 71.7)
- added R25: 13.3k, Resistor_SMD:R_0402_1005Metric, F.Cu at (180.9, 85.2)
- added R26: 1k, Resistor_SMD:R_0402_1005Metric, F.Cu at (174.4, 71.5)
- added R30: 13.3k, Resistor_SMD:R_0402_1005Metric, F.Cu at (180.9, 132.1)
- added R31: 13.3k, Resistor_SMD:R_0402_1005Metric, F.Cu at (180.9, 179.1)
- added R32: 13.3k, Resistor_SMD:R_0402_1005Metric, F.Cu at (180.9, 226.1)
- added R33: 13.3k, Resistor_SMD:R_0402_1005Metric, F.Cu at (174.3, 59.2)
- added R34: 1k, Resistor_SMD:R_0402_1005Metric, F.Cu at (161.0, 72.6)
- added R35: 1k, Resistor_SMD:R_0402_1005Metric, F.Cu at (161.0, 71.5)
- added R36: 1k, Resistor_SMD:R_0402_1005Metric, F.Cu at (148.9, 74.3)
- added REF**: EO silk 14mm, EO logos:EO silk 14mm, F.Cu at (145.9, 206.7)
- added REF**: OSHW-Logo2_14.6x12mm_SilkScreen, Symbol:OSHW-Logo2_14.6x12mm_SilkScreen, F.Cu at (162.2, 207.7)
- added REF**: EO silk 14mm, EO logos:EO silk 14mm, B.Cu at (193.5, 157.0)
- added REF**: OSHW-Logo2_14.6x12mm_SilkScreen, Symbol:OSHW-Logo2_14.6x12mm_SilkScreen, B.Cu at (176.1, 157.7)
- C10, C18, C4: value 10uf -> 22uf
- C11, C14, C28, C6: value 10uf -> .1uf; footprint Capacitor_SMD:C_1206_3216Metric -> Capacitor_SMD:C_0402_1005Metric
- C12, C13, C17, C23, C24, C27, C3, C34, C35, C5: footprint Capacitor_SMD:C_0603_1608Metric -> Capacitor_SMD:C_0402_1005Metric
- C15: value .1uf -> 56pf; footprint Capacitor_SMD:C_0603_1608Metric -> Capacitor_SMD:C_0402_1005Metric
- C16, C26, C8: value .1uf -> 22uf; footprint Capacitor_SMD:C_0603_1608Metric -> Capacitor_SMD:C_1206_3216Metric
- C19: value .1uf -> 10uf; footprint Capacitor_SMD:C_0603_1608Metric -> Capacitor_SMD:C_1206_3216Metric
- C2, C25: value 10uf -> 100uf; footprint Capacitor_SMD:C_1206_3216Metric -> Capacitor_SMD:CP_Elec_6.3x7.7; moved to B.Cu
- C7: value .1uf -> 75pf; footprint Capacitor_SMD:C_0603_1608Metric -> Capacitor_SMD:C_0402_1005Metric
- C9: value 100pf -> 22uf; footprint Capacitor_SMD:C_0603_1608Metric -> Capacitor_SMD:C_1206_3216Metric
- D1: value D -> SS34; footprint Package_TO_SOT_SMD:TO-252-3_TabPin2 -> Diode_SMD:D_SMA
- J5: value Conn_01x02_Pin -> 24v; footprint footprints:1x02_P5.00mm_Horizontal_terminal_block -> footprints:2x02_P3.5_KF2EDGSR; moved to F.Cu
- L1, L2: value 10uH -> 15uH; footprint Inductor_SMD:L_Taiyo-Yuden_MD-5050 -> footprints:CY54_INDUCTOR
- R1, R7: value 100k -> 500k; footprint Resistor_SMD:R_0603_1608Metric -> Resistor_SMD:R_0402_1005Metric
- R2: value 158k -> 100k; footprint Resistor_SMD:R_0603_1608Metric -> Resistor_SMD:R_0402_1005Metric
- R3, R6: value 30.1k -> 100k; footprint Resistor_SMD:R_0603_1608Metric -> Resistor_SMD:R_0402_1005Metric
- R4: value 100k -> 13.3k; footprint Resistor_SMD:R_0603_1608Metric -> Resistor_SMD:R_0402_1005Metric
- R5: value 158K -> 500k; footprint Resistor_SMD:R_0603_1608Metric -> Resistor_SMD:R_0402_1005Metric
- R8: value 93.1k -> 100k; footprint Resistor_SMD:R_0603_1608Metric -> Resistor_SMD:R_0402_1005Metric
- R9: value 30.1k -> 22.1k; footprint Resistor_SMD:R_0603_1608Metric -> Resistor_SMD:R_0402_1005Metric
- U1: value AP63201WU -> TPS54202DDC; footprint Package_TO_SOT_SMD:TSOT-23-6 -> Package_TO_SOT_SMD:SOT-23-6
- U2, U25: value AOZ1360AIL -> TPS54202DDC; footprint footprints:AOZ1360AIL_AOS -> Package_TO_SOT_SMD:SOT-23-6
- moved C10 43.8 mm to (186.6, 61.0)
- moved C11 39.6 mm to (183.2, 62.5), turned to 0 degrees
- moved U2 38.3 mm to (182.1, 64.8)
- moved C27 36.7 mm to (156.3, 62.5)
- moved C28 36.0 mm to (153.9, 67.0), turned to 0 degrees
- moved U25 35.1 mm to (155.2, 64.8), turned to 180 degrees
- moved C4 34.2 mm to (173.1, 60.9)
- moved C16 32.3 mm to (187.2, 69.6), turned to 180 degrees
- moved R1 31.7 mm to (169.8, 61.5), turned to 0 degrees
- moved C5 31.6 mm to (169.8, 62.5), turned to 0 degrees
- moved R7 30.4 mm to (156.3, 61.5), turned to 0 degrees
- moved C9 29.7 mm to (169.1, 69.5), turned to 0 degrees
- moved R2 28.6 mm to (167.6, 61.5), turned to 180 degrees
- moved C26 26.8 mm to (159.6, 61.0), turned to 180 degrees
- moved C8 26.0 mm to (173.8, 69.5)
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Connections:
- C10 pad 1: +5V -> GND
- C10 pad 2: GND -> +24V
- C11 pad 1: +5V -> GND
- C11 pad 2: GND -> +24V
- C14 pad 1: +24V -> Net-(U2-BOOT)
- C14 pad 2: GND -> Net-(U2-SW)
- C15 pad 1: Net-(U23-SS) -> Net-(U2-FB)
- C15 pad 2: GND -> +3.3VA
- C16 pad 1: Net-(U24-EN) -> GND
- C16 pad 2: GND -> +3.3VA
- C18 pad 1: Net-(U24-EN) -> GND
- C18 pad 2: GND -> +3.3VA
- C19 pad 1: Net-(U24-SW) -> +24V
- C19 pad 2: Net-(U24-BST) -> GND
- C26 pad 1: Net-(U25-SS) -> GND
- C26 pad 2: GND -> +24V
- C27 pad 1: SLOT A 24V -> GND
- C27 pad 2: GND -> +24V
- C28 pad 1: SLOT A 24V -> Net-(U25-BOOT)
- C28 pad 2: GND -> Net-(U25-SW)
- C4 pad 1: Net-(U1-EN) -> GND
- C4 pad 2: GND -> +24V
- C5 pad 1: Net-(U1-EN) -> GND
- C5 pad 2: GND -> +24V
- C6 pad 1: +24V -> Net-(U1-BOOT)
- C6 pad 2: GND -> Net-(U1-SW)
- C7 pad 1: Net-(U2-SS) -> Net-(U1-FB)
- C7 pad 2: GND -> +5VA
- C8 pad 1: Net-(U1-SW) -> GND
- C8 pad 2: Net-(U1-BST) -> +5VA
- C9 pad 1: +5V -> GND
- C9 pad 2: Net-(U1-FB) -> +5VA
- J1 pad P$A10: +3.3VP -> +3.3VA
- J1 pad P$A11: +5VP -> +5VA
- J1 pad P$B10: +3.3VP -> +3.3VA
- J1 pad P$B11: +5VP -> +5VA
- J2 pad P$A1: SLOT A 24V -> SLOT B 24V
- J2 pad P$A10: +3.3VP -> +3.3VA
- J2 pad P$A11: +5VP -> +5VA
- J2 pad P$A2: SLOT A 24V -> SLOT B 24V
- J2 pad P$A3: SLOT A 24V -> SLOT B 24V
- J2 pad P$A4: SLOT A 24V -> SLOT B 24V
- J2 pad P$B1: SLOT A 24V -> SLOT B 24V
- J2 pad P$B10: +3.3VP -> +3.3VA
- J2 pad P$B11: +5VP -> +5VA
- J2 pad P$B2: SLOT A 24V -> SLOT B 24V
- J2 pad P$B3: SLOT A 24V -> SLOT B 24V
- J2 pad P$B4: SLOT A 24V -> SLOT B 24V
- J3 pad P$A1: SLOT A 24V -> SLOT C 24V
- J3 pad P$A10: +3.3VP -> +3.3VA
- J3 pad P$A11: +5VP -> +5VA
- J3 pad P$A2: SLOT A 24V -> SLOT C 24V
- J3 pad P$A3: SLOT A 24V -> SLOT C 24V
- J3 pad P$A4: SLOT A 24V -> SLOT C 24V
- J3 pad P$B1: SLOT A 24V -> SLOT C 24V
- J3 pad P$B10: +3.3VP -> +3.3VA
- J3 pad P$B11: +5VP -> +5VA
- J3 pad P$B2: SLOT A 24V -> SLOT C 24V
- J3 pad P$B3: SLOT A 24V -> SLOT C 24V
- J3 pad P$B4: SLOT A 24V -> SLOT C 24V
- J4 pad P$A1: SLOT A 24V -> SLOT D 24V
- J4 pad P$A10: +3.3VP -> +3.3VA
- J4 pad P$A11: +5VP -> +5VA
- J4 pad P$A2: SLOT A 24V -> SLOT D 24V
- J4 pad P$A3: SLOT A 24V -> SLOT D 24V
- J4 pad P$A4: SLOT A 24V -> SLOT D 24V
- J4 pad P$B1: SLOT A 24V -> SLOT D 24V
- J4 pad P$B10: +3.3VP -> +3.3VA
- J4 pad P$B11: +5VP -> +5VA
- J4 pad P$B2: SLOT A 24V -> SLOT D 24V
- J4 pad P$B3: SLOT A 24V -> SLOT D 24V
- J4 pad P$B4: SLOT A 24V -> SLOT D 24V
- J5 pad 2: GND -> Net-(J5-Pin_1)
- L1 pad 2: +5V -> +5VA
- L2 pad 1: Net-(U24-SW) -> Net-(U2-SW)
- L2 pad 2: +5VP -> +3.3VA
- R1 pad 1: Net-(U2-SET) -> Net-(U1-EN)
- R1 pad 2: GND -> +24V
- R2 pad 1: Net-(U1-FB) -> GND
- R2 pad 2: +5V -> Net-(U1-EN)
- R3 pad 1: GND -> Net-(U1-FB)
- R3 pad 2: Net-(U1-FB) -> +5VA
- R4 pad 1: Net-(U23-SET) -> GND
- R4 pad 2: GND -> Net-(U1-FB)
- R5 pad 1: Net-(U24-FB) -> Net-(U2-EN)
- R5 pad 2: +5VP -> +24V
- R6 pad 2: Net-(U24-FB) -> Net-(U2-EN)
- R7 pad 1: Net-(U25-SET) -> Net-(U25-EN)
- R7 pad 2: GND -> +24V
- R8 pad 1: Net-(U26-FB) -> Net-(U2-FB)
- R8 pad 2: +3.3VP -> +3.3VA
- R9 pad 2: Net-(U26-FB) -> Net-(U2-FB)
- U1 pad 1: Net-(U1-FB) -> GND
- U1 pad 2: Net-(U1-EN) -> Net-(U1-SW)
- U1 pad 3: Net-(U1-EN) -> +24V
- U1 pad 4: GND -> Net-(U1-FB)
- U1 pad 5: Net-(U1-SW) -> Net-(U1-EN)
- U1 pad 6: Net-(U1-BST) -> Net-(U1-BOOT)
- U2 pad 1: +24V -> GND
- U2 pad 2: +24V -> Net-(U2-SW)
- U2 pad 3: GND -> +24V
- U2 pad 4: Net-(U2-SS) -> Net-(U2-FB)
- U2 pad 5: +24V -> Net-(U2-EN)
- U2 pad 6: Net-(U2-SET) -> Net-(U2-BOOT)
- U25 pad 1: +24V -> GND
- U25 pad 2: +24V -> Net-(U25-SW)
- U25 pad 3: GND -> +24V
- U25 pad 4: Net-(U25-SS) -> Net-(U25-FB)
- U25 pad 5: +24V -> Net-(U25-EN)
- U25 pad 6: Net-(U25-SET) -> Net-(U25-BOOT)
Routing:
- net SLOT A 24V: track 51.9 -> 16.4 mm, vias 32 -> 8
- net Net-(U24-EN): track 28.9 -> 0.00 mm, vias 8 -> 0
- net +5VA: track 0.00 -> 21.5 mm, vias 0 -> 9
- net +24V: track 91.1 -> 70.3 mm, vias 9 -> 7
- net +3.3VA: track 0.00 -> 20.6 mm, vias 0 -> 9
- net +5VP: track 20.2 -> 0.00 mm, vias 8 -> 0
- net +3.3VP: track 20.2 -> 0.00 mm, vias 8 -> 0
- net SLOT C 24V: track 0.00 -> 16.7 mm, vias 0 -> 8
- net SLOT B 24V: track 0.00 -> 16.7 mm, vias 0 -> 8
- net SLOT D 24V: track 0.00 -> 16.5 mm, vias 0 -> 8
- net GND: track 331.2 -> 316.4 mm, vias 221 -> 292
- net Net-(U24-FB): track 9.99 -> 0.00 mm
- net Net-(U26-FB): track 9.64 -> 0.00 mm
- net Net-(U25-FB): track 0.00 -> 7.94 mm, vias 0 -> 2
- net Net-(U2-FB): track 0.00 -> 7.94 mm, vias 0 -> 2
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- added copper zone on B.Cu, net +24V
- added copper zone on F.Cu, net +3.3VA
- added copper zone on F.Cu, net +5VA
- added copper zone on B.Cu, net GND
- added copper zone on F.Cu, net Net-(U2-SW)
- added copper zone on F.Cu, net Net-(U25-SW)
- added copper zone on F.Cu, net SLOT B 24V
- added copper zone on F.Cu, net SLOT C 24V
- added copper zone on F.Cu, net SLOT D 24V
- removed copper zone on F.Cu, net +3.3VP
- removed copper zone on F.Cu, net +5VP
- removed copper zone on F.Cu, net Net-(U1-EN)
- removed copper zone on F.Cu, net Net-(U24-EN)
- removed copper zone on F.Cu, net Net-(U24-SW)
- removed copper zone on F.Cu, net Net-(U26-SW)
Other:
- outline, holes or cut-outs redrawn
- board text added: "- +"
- board text added: "BOARD 24v"
- board text added: "BP-1"
- board text added: "MYIR Z-TURN V2"
- board text added: "REV 0.1"
- board text added: "SLOT 3.3v"
- board text added: "SLOT 5v"
- board text added: "SLOTA 24v"
- board text added: "SLOTB 24v"
- board text added: "SLOTC 24v"
- board text added: "SLOTD 24v"
- board text added: "ZYNQ 3.3v"
- board text added: "ZYNQ 5v"
