File: KiCad/Motion controller MiYR interface/Motion controller MiYR interface.kicad_sch (KiCad schematic)
At the start: 136 parts, among them CN1 Conn_02x40_Odd_Even, CN2 Conn_02x40_Odd_Even, J1 10061913-111PLF, J2 10061913-111PLF, J3 10061913-111PLF, J4 10061913-111PLF, J5 Conn_01x02_Pin, U1 AP63201WU, U10 D1213A-04S-7, U11 D1213A-04S-7, U12 D1213A-04S-7, U13 D1213A-04S-7, U14 D1213A-04S-7, U15 D1213A-04S-7, U16 D1213A-04S-7, U17 D1213A-04S-7, U18 D1213A-04S-7, U19 D1213A-04S-7, U2 AOZ1360AIL, U20 D1213A-04S-7, U21 D1213A-04S-7, U22 D1213A-04S-7, U23 AOZ1360AIL, U24 AP63201WU, U25 AOZ1360AIL, U26 AP63201WU, U3 D1213A-04S-7, U30 D1213A-04S-7, U31 D1213A-04S-7, U32 D1213A-04S-7, U33 D1213A-04S-7, U34 74HC165, U35 74HC595, U36 LM324, U37 LM324, U4 D1213A-04S-7, U5 D1213A-04S-7, U6 D1213A-04S-7, U7 D1213A-04S-7, U8 D1213A-04S-7, U9 D1213A-04S-7

Commit message: update
Parts:
- removed C2, C21, C22, C25, C29, C32, C33: 10uf, Capacitor_SMD:C_1206_3216Metric, symbol Device:C
- removed C20, C31: 100pf, Capacitor_SMD:C_0603_1608Metric, symbol Device:C
- removed C30: .1uf, Capacitor_SMD:C_0603_1608Metric, symbol Device:C
- removed C49, C51: .1uf, symbol Device:C
- removed D1: D, Package_TO_SOT_SMD:TO-252-3_TabPin2, symbol Device:D
- removed J5: Conn_01x02_Pin, footprints:1x02_P5.00mm_Horizontal_terminal_block, symbol Connector:Conn_01x02_Pin
- removed L3: 6.8uH, Inductor_SMD:L_Taiyo-Yuden_MD-5050, symbol Device:L
- removed R1, R15, R4, R7: 100k, Resistor_SMD:R_0603_1608Metric, symbol Device:R
- removed R17, R18, R19, R24, R25, R26, R30, R31, R32, R36, R37, R38, R42, R43, R44, R45, R46, R47, R48, R49, R50, R51, R52, R53, R54, R55: 10k, symbol Device:R
- removed R2: 158k, Resistor_SMD:R_0603_1608Metric, symbol Device:R
- removed R20, R21, R22, R23, R27, R28, R29, R33, R34, R35, R39, R40, R41, R57, R61: 100k, symbol Device:R
- removed R3, R6, R9: 30.1k, Resistor_SMD:R_0603_1608Metric, symbol Device:R
- removed R5: 158K, Resistor_SMD:R_0603_1608Metric, symbol Device:R
- removed R8: 93.1k, Resistor_SMD:R_0603_1608Metric, symbol Device:R
- removed U1, U24, U26: AP63201WU, Package_TO_SOT_SMD:TSOT-23-6, symbol Regulator_Switching:AP63201WU
- removed U2, U23, U25: AOZ1360AIL, footprints:AOZ1360AIL_AOS, symbol AOZ1360AIL:AOZ1360AIL
- removed U34: 74HC165, symbol 74xx:74HC165
- removed U35: 74HC595, symbol 74xx:74HC595
- removed U36, U37: LM324, symbol Amplifier_Operational:LM324
- added C2, C25: 100uf, Capacitor_SMD:CP_Elec_6.3x7.7, symbol Device:C_Polarized_US
- added C36: 75pf, Capacitor_SMD:C_0402_1005Metric, symbol Device:C
- added C37, C38, C70, C72, C74: 22uf, Capacitor_SMD:C_1206_3216Metric, symbol Device:C
- added D1, D18, D19, D20, D21, D22: SS34, Diode_SMD:D_SMA, symbol Diode:SS34
- added D10, D11, D12, D13, D14, D15, D16, D2, D3: LED, LED_SMD:LED_0603_1608Metric, symbol Device:LED
- added F2, F3, F4, F5: 3A, Fuse:Fuse_2920_7451Metric, symbol Device:Polyfuse
- added H1, H10, H2, H3, H4, H5, H6, H7, H8, H9: MountingHole, MountingHole:MountingHole_3.2mm_M3, symbol Mechanical:MountingHole
- added J5: 24v, footprints:2x02_P3.5_KF2EDGSR, symbol Connector:Conn_01x04_Pin
- added L4: 15uH, footprints:CY54_INDUCTOR, symbol Device:L
- added M1, M2: Fan, Connector_PinHeader_2.54mm:PinHeader_1x02_P2.54mm_Vertical, symbol Motor:Fan
- added R1, R5, R7: 560k, Resistor_SMD:R_0402_1005Metric, symbol Device:R_US
- added R10, R11, R2, R3, R6, R8: 100k, Resistor_SMD:R_0402_1005Metric, symbol Device:R_US
- added R12, R25, R30, R31, R32, R33, R4: 13.3k, Resistor_SMD:R_0402_1005Metric, symbol Device:R_US
- added R17, R18, R26, R34, R35, R36: 1k, Resistor_SMD:R_0402_1005Metric, symbol Device:R_US
- added R9: 22.1k, Resistor_SMD:R_0402_1005Metric, symbol Device:R_US
- added U1, U2, U25: TPS54202DDC, Package_TO_SOT_SMD:SOT-23-6, symbol Regulator_Switching:TPS54202DDC
- C1, C10, C18, C4: value 10uf -> 22uf; Generic Allowed? (none) -> yes; LCSC# (none) -> C12891; Manufacturer (none) -> Samsung Electro-Mechanics; Part Number (none) -> CL31A226KAHNNNE; cost (none) -> 0.04
- C11, C14, C28, C6: value 10uf -> .1uf; footprint Capacitor_SMD:C_1206_3216Metric -> Capacitor_SMD:C_0402_1005Metric; Generic Allowed? (none) -> yes; LCSC# (none) -> C105882; Manufacturer (none) -> YAGEO; Part Number (none) -> CC0402KRX5R9BB104; cost (none) -> 0.003
- C12, C13, C17, C23, C24, C27, C3, C34, C35, C5: footprint Capacitor_SMD:C_0603_1608Metric -> Capacitor_SMD:C_0402_1005Metric; Generic Allowed? (none) -> yes; LCSC# (none) -> C105882; Manufacturer (none) -> YAGEO; Part Number (none) -> CC0402KRX5R9BB104; cost (none) -> 0.003
- C15: value .1uf -> 56pf; footprint Capacitor_SMD:C_0603_1608Metric -> Capacitor_SMD:C_0402_1005Metric; Generic Allowed? (none) -> yes; LCSC# (none) -> C107007; Manufacturer (none) -> YAGEO; Part Number (none) -> CC0402JRNPO9BN560; cost (none) -> 0.0011
- C16, C19, C26, C8: value .1uf -> 22uf; footprint Capacitor_SMD:C_0603_1608Metric -> Capacitor_SMD:C_1206_3216Metric; Generic Allowed? (none) -> yes; LCSC# (none) -> C12891; Manufacturer (none) -> Samsung Electro-Mechanics; Part Number (none) -> CL31A226KAHNNNE; cost (none) -> 0.04
- C48, C50: value .1uf -> 22uf; footprint (none) -> Capacitor_SMD:C_1206_3216Metric; Generic Allowed? (none) -> yes; LCSC# (none) -> C12891; Manufacturer (none) -> Samsung Electro-Mechanics; Part Number (none) -> CL31A226KAHNNNE; cost (none) -> 0.04
- C7: value .1uf -> 75pf; footprint Capacitor_SMD:C_0603_1608Metric -> Capacitor_SMD:C_0402_1005Metric; Generic Allowed? (none) -> yes; LCSC# (none) -> C107010; Manufacturer (none) -> YAGEO; Part Number (none) -> CC0402JRNPO9BN750; cost (none) -> 0.0011
- C9: value 100pf -> 22uf; footprint Capacitor_SMD:C_0603_1608Metric -> Capacitor_SMD:C_1206_3216Metric; Generic Allowed? (none) -> yes; LCSC# (none) -> C12891; Manufacturer (none) -> Samsung Electro-Mechanics; Part Number (none) -> CL31A226KAHNNNE; cost (none) -> 0.04
- CN1, CN2: Generic Allowed? (none) -> yes; LCSC# (none) -> C45359092; Manufacturer (none) -> HDGC; Part Number (none) -> HDGC127-PS2-40; cost (none) -> 0.44
- F1: Generic Allowed? (none) -> yes, 35vdc+; LCSC# (none) -> C136354; Manufacturer (none) -> JDTfuse; Part Number (none) -> JFC1206-2100FS; cost (none) -> 0.065
- J1, J2, J3, J4: Generic Allowed? (none) -> yes; LCSC# (none) -> C48985837; Manufacturer (none) -> UMAX; Part Number (none) -> 3113-111P; cost (none) -> 0.85
- L1, L2: value 10uH -> 15uH; footprint Inductor_SMD:L_Taiyo-Yuden_MD-5050 -> footprints:CY54_INDUCTOR; Generic Allowed? (none) -> yes; LCSC# (none) -> C2929432; Manufacturer (none) -> SHOU HAN; Part Number (none) -> CY54-15UH; cost (none) -> 0.05
- U10, U11, U12, U13, U14, U15, U16, U17, U18, U19, U20, U21, U22, U3, U30, U31, U32, U33, U4, U5, U6, U7, U8, U9: value D1213A-04S-7 -> ESLC0504F; Generic Allowed? (none) -> yes; LCSC# (none) -> C42385170; Manufacturer (none) -> ElecSuper; Part Number (none) -> ESLC0504F; cost (none) -> 0.065
Connections:
- net +24V: now also C10.2, C11.2, C19.1, C26.2, C27.2, C4.2, C5.2, C2.1, C25.1, C74.1, D1.1 (K), D14.2 (A), D18.1 (K), F2.1, F3.1, F4.1, F5.1, M1.1 (+), M2.1 (+), R1.2, R5.2, R7.2, U1.3 (VIN), U2.3 (VIN), U25.3 (VIN); no longer C14.1, C6.1
- net +3.3V: now also D16.2 (A); no longer C48.1, C50.1
- net +5V: now also C36.2, C37.2, C38.2, D15.2 (A), L4.2, R11.2; no longer C10.1, C11.1, C9.1, L1.2
- net GND: now also C10.1, C11.1, C16.1, C18.1, C19.2, C26.1, C27.1, C4.1, C5.1, C8.1, C9.1, C2.2, C25.2, C37.1, C38.1, C70.2, C72.2, C74.2, D1.2 (A), D18.2 (A), D19.2 (A), D20.2 (A), D21.2 (A), D22.2 (A), J5.3 (Pin_3), J5.4 (Pin_4), M1.2 (-), M2.2 (-), R10.1, R12.1, R18.1, R2.1, R25.1, R26.1, R30.1, R31.1, R32.1, R33.1, R35.1, R36.1, R4.1, R6.1, R9.1, U1.1 (GND), U2.1 (GND), U25.1 (GND); no longer C10.2, C11.2, C14.2, C15.2, C16.2, C18.2, C26.2, C27.2, C28.2, C4.2, C5.2, C6.2, C7.2
- net SLOT A 24V: now also C48.1, D10.2 (A), D19.1 (K), F2.2; no longer C27.1, C28.1, J2.P$A1 (A1), J2.P$A2 (A2), J2.P$A3 (A3), J2.P$A4 (A4), J2.P$B1 (B1), J2.P$B2 (B2), J2.P$B3 (B3), J2.P$B4 (B4), J3.P$A1 (A1), J3.P$A2 (A2), J3.P$A3 (A3), J3.P$A4 (A4), J3.P$B1 (B1), J3.P$B2 (B2), J3.P$B3 (B3), J3.P$B4 (B4), J4.P$A1 (A1), J4.P$A2 (A2), J4.P$A3 (A3), J4.P$A4 (A4), J4.P$B1 (B1), J4.P$B2 (B2), J4.P$B3 (B3), J4.P$B4 (B4)
- net at L1.1: now also C6.2, U1.2 (SW); no longer C8.1
- net +5VA: now reaches C8.2
- net +5VA: now also C7.2, C9.2, J1.P$A11 (A11), J1.P$B11 (B11), J2.P$A11 (A11), J2.P$B11 (B11), J3.P$A11 (A11), J3.P$B11 (B11), J4.P$A11 (A11), J4.P$B11 (B11), L1.2, D2.2 (A), R3.2
- net at C15.1: now also R8.1, R9.2, U2.4 (FB)
- net at F1.1: now also J5.1 (Pin_1), J5.2 (Pin_2)
- net at L2.1: now also C14.2, U2.2 (SW); no longer C19.1
- net at C7.1: now also R3.1, R4.2, U1.4 (FB)
- net +3.3VP renamed +3.3VA
- net +3.3VA: now also C15.2, C16.2, C18.2, L2.2, D3.2 (A), R8.2
- removed net +5VP: J1.P$A11 (A11), J1.P$B11 (B11), J2.P$A11 (A11), J2.P$B11 (B11), J3.P$A11 (A11), J3.P$B11 (B11), J4.P$A11 (A11), J4.P$B11 (B11), L2.2
- new net: D10.1 (K), R25.2
- new net: C36.1, R11.1, R12.2, U25.4 (FB)
- new net: C6.1, U1.6 (BOOT)
- new net: D3.1 (K), R18.2
- new net: R10.2, R7.1, U25.5 (EN)
- new net: D13.1 (K), R32.2
- new net: D2.1 (K), R17.2
- new net: D15.1 (K), R34.2
- new net: D11.1 (K), R30.2
- new net: R17.1, R26.2
- new net: D16.1 (K), R36.2
- new net: D12.1 (K), R31.2
- new net: R34.1, R35.2
- new net: C28.1, U25.6 (BOOT)
- new net: C28.2, L4.1, U25.2 (SW)
- new net: R1.1, R2.2, U1.5 (EN)
- new net: D14.1 (K), R33.2
- new net: R5.1, R6.2, U2.5 (EN)
- new net: C14.1, U2.6 (BOOT)
- new net SLOT B 24V: C50.1, D11.2 (A), D20.1 (K), F3.2, J2.P$A1 (A1), J2.P$A2 (A2), J2.P$A3 (A3), J2.P$A4 (A4), J2.P$B1 (B1), J2.P$B2 (B2), J2.P$B3 (B3), J2.P$B4 (B4)
- new net SLOT C 24V: C70.1, D12.2 (A), D21.1 (K), F4.2, J3.P$A1 (A1), J3.P$A2 (A2), J3.P$A3 (A3), J3.P$A4 (A4), J3.P$B1 (B1), J3.P$B2 (B2), J3.P$B3 (B3), J3.P$B4 (B4)
- new net SLOT D 24V: C72.1, D13.2 (A), D22.1 (K), F5.2, J4.P$A1 (A1), J4.P$A2 (A2), J4.P$A3 (A3), J4.P$A4 (A4), J4.P$B1 (B1), J4.P$B2 (B2), J4.P$B3 (B3), J4.P$B4 (B4)
Other:
- note added: "SLOT POWER"
- note added: "ZYNQ 5V BUCK CONVERTER"
- note removed: "1.65v ref"
- note removed: "2.18v ref"
- note removed: "SLOT 24V SOFT START AND CURRENT LIMIT (4A)"
- note removed: "SLOT 3.3V BUCK CONVERTER"
- note removed: "SLOT 5V/3.3V SOFT START AND BUCK CONVERTER"
- note removed: "ZYNQ 5V SOFT START AND BUCK CONVERTER"
- note removed: "trip level ~18v"
- moved on the sheet: F1, U10, U11, U12, U13, U14, U15, U16, U17, U18, U19, U20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
