File: KiCad/Mezzanine jumper/Mezzanine jumper.kicad_pcb (KiCad board)
At the start: 4 copper layers, 33 x 34.5 mm, 6 parts, among them J1 BB0500100M-1002C-001, J2 BB0500100M-1002C-001

Commit message: fix jumper
Routing:
- net /IO_38: track 27.8 -> 28.3 mm
- net /IO_39: track 27.0 -> 27.5 mm
- net /IO_46: track 27.8 -> 28.3 mm
- net /IO_22: track 27.8 -> 28.3 mm
- net /IO_14: track 27.8 -> 28.3 mm
- net /IO_47: track 27.0 -> 27.5 mm
- net /IO_45: track 27.0 -> 26.5 mm
- net /IO_37: track 27.0 -> 26.5 mm
- net /IO_31: track 27.0 -> 27.5 mm
- net /IO_30: track 27.8 -> 28.3 mm
- net /IO_29: track 27.0 -> 26.5 mm
- net /IO_23: track 27.0 -> 27.5 mm
- net /IO_21: track 27.0 -> 26.5 mm
- net /IO_20: track 27.8 -> 27.3 mm
- net /IO_15: track 27.0 -> 27.5 mm
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
Commit message: update
Other:
- board text added: "commit: 7a841bd"
- board text removed: "commit: xxx"
