File: KiCad/16x Card Module/FPGA_Connector.kicad_sch (KiCad schematic)
At the start: 9 parts, among them J1 Conn_02x25_Odd_Even, U2 D1213A-04S-7, U3 D1213A-04S-7, U4 D1213A-04S-7, U5 D1213A-04S-7, U6 D1213A-04S-7

Commit message: update
Parts:
- J1: LCSC# (none) -> C2883281; Manufacturer (none) -> XKB Connection; Part Number (none) -> X4621WR-2x25I-C40D28
Changed lines of the file:
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@@
+			)
+		)
+		(property "LCSC#" "C2883281"
+			(at 48.26 67.31 0)
+			(effects
+				(font
+					(size 1.27 1.27)
+				)
+				(hide yes)
+			)
+		)
+		(property "Manufacturer" "XKB Connection"
+			(at 48.26 67.31 0)
+			(effects
+				(font
+					(size 1.27 1.27)
+				)
+				(hide yes)
+			)
+		)
+		(property "Part Number" "X4621WR-2x25I-C40D28"
+			(at 48.26 67.31 0)
+			(effects
+				(font
+					(size 1.27 1.27)
+				)
+				(hide yes)
 			)
 		)
