File: KiCad/Mezzanine Backplane/Mezzanine Backplane.kicad_sch (KiCad schematic)
At the start: 4 parts, among them J1 BB0500220F-1002C-001, J2 BB0500220F-1002C-001, J3 Conn_02x25_Odd_Even, J4 Conn_02x25_Odd_Even

Commit message: update
Parts:
- J3, J4: LCSC# (none) -> C42163108; Manufacturer (none) -> Hong Cheng; Part Number (none) -> HC-PM200-4.3H-2x25PS
Changed lines of the file:
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@@
+			)
+		)
+		(property "LCSC#" "C42163108"
+			(at 149.86 114.3 0)
+			(effects
+				(font
+					(size 1.27 1.27)
+				)
+				(hide yes)
+			)
+		)
+		(property "Manufacturer" "Hong Cheng"
+			(at 149.86 114.3 0)
+			(effects
+				(font
+					(size 1.27 1.27)
+				)
+				(hide yes)
+			)
+		)
+		(property "Part Number" "HC-PM200-4.3H-2x25PS"
+			(at 149.86 114.3 0)
+			(effects
+				(font
+					(size 1.27 1.27)
+				)
+				(hide yes)
 			)
 		)
@@
 			(at 234.95 114.3 0)
 			(effects
+				(font
+					(size 1.27 1.27)
+				)
+				(hide yes)
+			)
+		)
+		(property "LCSC#" "C42163108"
+			(at 234.95 114.3 0)
+			(effects
+				(font
+					(size 1.27 1.27)
+				)
+				(hide yes)
+			)
+		)
+		(property "Manufacturer" "Hong Cheng"
+			(at 234.95 114.3 0)
+			(effects
+				(font
+					(size 1.27 1.27)
+				)
+				(hide yes)
+			)
+		)
+		(property "Part Number" "HC-PM200-4.3H-2x25PS"
+			(at 234.95 114.3 0)
+			(effects
