File: KiCad/Mezzanine Jumper up16/Mezzanine Jumper up16.kicad_pcb (KiCad board)
At the start: 4 copper layers, 33 x 34.5 mm, 6 parts, among them J1 BB0500100M-1002C-001, J2 BB0500100M-1002C-001

Commit message: update
Other:
- board text added: "commit: 7a841bd"
- board text removed: "commit: xxx"
