File: KiCad/Modular MiYR interface/Modular MiYR interface.kicad_pcb (KiCad board)
At the start: 4 copper layers, 65.5 x 107 mm, 86 parts, among them CN1 Conn_02x40_Odd_Even, CN2 Conn_02x40_Odd_Even, J1 FPC-05FB-50PH20, J2 FPC-05FB-50PH20, J3 FPC-05FB-50PH20, J4 FPC-05FB-50PH20, J5 FPC-05FB-50PH20, J6 24v, J7 Conn_01x08_Socket, M1 Fan, U1 TPS54202DDC, U2 TPS54202DDC, U3 TPS54202DDC

Commit message: fix jumper
Other:
- board text added: "commit: de769dd"
- board text removed: "commit: xxx"
Changed lines of the file:
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@@
 			(psa4output no)
 			(plotreference yes)
-			(plotvalue yes)
+			(plotvalue no)
 			(plotfptext yes)
 			(plotinvisibletext no)
@@
 			(outputformat 1)
 			(mirror no)
-			(drillshape 1)
+			(drillshape 0)
 			(scaleselection 1)
-			(outputdirectory "")
+			(outputdirectory "manufacturing outputs/")
 		)
 	)
@@
 		)
 	)
-	(gr_text "commit: xxx"
+	(gr_text "commit: de769dd"
 		(at 82.5 99.4 90)
 		(layer "B.SilkS")
