File: KiCad/Main Mezzanine Backplane/Main Mezzanine Backplane.kicad_pcb (KiCad board)
At the start: 4 copper layers, 48 x 97 mm, 42 parts, among them J1 BB0500220F-1002C-001, J2 BB0500220F-1002C-001, J3 FPC-05FB-50PH20, J4 FPC-05FB-50PH20, J5 FPC-05FB-50PH20, J6 FPC-05FB-50PH20, J7 FPC-05FB-50PH20, U1 D1213A-04S-7, U10 D1213A-04S-7, U11 D1213A-04S-7, U12 D1213A-04S-7, U13 D1213A-04S-7, U14 D1213A-04S-7, U15 D1213A-04S-7, U16 D1213A-04S-7, U17 D1213A-04S-7, U18 D1213A-04S-7, U19 D1213A-04S-7, U2 D1213A-04S-7, U20 D1213A-04S-7, U21 D1213A-04S-7, U22 D1213A-04S-7, U23 D1213A-04S-7, U24 D1213A-04S-7, U25 D1213A-04S-7, U26 D1213A-04S-7, U3 D1213A-04S-7, U4 D1213A-04S-7, U5 D1213A-04S-7, U6 D1213A-04S-7, U7 D1213A-04S-7, U8 D1213A-04S-7, U9 D1213A-04S-7

Commit message: update serial module and backplane hw
Connections:
- J3 pad 10: GND -> unconnected-(J3-Pad10)
- J3 pad 18: +5V -> GND
- J3 pad 19: +5V -> +3.3V
- J3 pad 20: +5V -> +3.3V
- J3 pad 21: +5V -> +3.3V
- J3 pad 22: +5V -> +3.3V
- J3 pad 23: GND -> +3.3V
- J3 pad 28: +3.3V -> GND
- J3 pad 29: +3.3V -> +5V
- J3 pad 30: +3.3V -> +5V
- J3 pad 31: +3.3V -> +5V
- J3 pad 32: +3.3V -> +5V
- J3 pad 33: GND -> +5V
- J3 pad 41: unconnected-(J3-Pad41) -> GND
- J3 pad 42: +24V -> unconnected-(J3-Pad42)
- J3 pad 9: unconnected-(J3-Pad9) -> +24V
Routing:
- net +5V: track 172.5 -> 182.6 mm
- net GND: track 223.7 -> 222.6 mm, vias 462 -> 469
- net +24V: track 64.1 -> 64.8 mm
Other:
- board text added: "commit:"
- board text removed: "commit: de769dd"
