File: KiCad/Main Mezzanine Backplane/Main Mezzanine Backplane.kicad_sch (KiCad schematic)
At the start: 11 parts, among them J1 BB0500220F-1002C-001, J2 BB0500220F-1002C-001, J3 FPC-05FB-50PH20, J4 FPC-05FB-50PH20, J5 FPC-05FB-50PH20, J6 FPC-05FB-50PH20, J7 FPC-05FB-50PH20

Commit message: update serial module and backplane hw
Connections:
- net +24V: now also J3.9; no longer J3.42
- net +3.3V: now also J3.19, J3.20, J3.21, J3.22, J3.23; no longer J3.28, J3.29, J3.30, J3.31, J3.32
- net +5V: now also J3.29, J3.30, J3.31, J3.32, J3.33; no longer J3.18, J3.19, J3.20, J3.21, J3.22
- net GND: now also J3.18, J3.28, J3.41; no longer J3.10, J3.23, J3.33
