File: KiCad/Serial Module/FPGA_Connector.kicad_sch (KiCad schematic)
At the start: 9 parts, among them J1 Conn_02x25_Odd_Even, U2 D1213A-04S-7, U3 D1213A-04S-7, U4 D1213A-04S-7, U5 D1213A-04S-7, U6 D1213A-04S-7

Commit message: update serial module and backplane hw
Parts:
- U2, U3, U4, U5: now fitted
Connections:
- net IO_0: now also J1.3 (Pin_3)
- net IO_1: now also J1.5 (Pin_5)
- net IO_10: now also J1.25 (Pin_25)
- net IO_11: now also J1.27 (Pin_27)
- net IO_12: now also J1.31 (Pin_31)
- net IO_13: now also J1.33 (Pin_33)
- net IO_14: now also J1.35 (Pin_35)
- net IO_15: now also J1.37 (Pin_37)
- net IO_2: now also J1.7 (Pin_7)
- net IO_3: now also J1.9 (Pin_9)
- net IO_4: now also J1.11 (Pin_11)
- net IO_5: now also J1.13 (Pin_13)
- net IO_6: now also J1.17 (Pin_17)
- net IO_7: now also J1.19 (Pin_19)
- net IO_8: now also J1.21 (Pin_21)
- net IO_9: now also J1.23 (Pin_23)
- net IN_0 renamed OUT_0
- net OUT_0: no longer J1.3 (Pin_3)
- net IN_1 renamed OUT_1
- net OUT_1: no longer J1.5 (Pin_5)
- net IN_10 renamed OUT_10
- net OUT_10: no longer J1.25 (Pin_25)
- net IN_11 renamed OUT_11
- net OUT_11: no longer J1.27 (Pin_27)
- net IN_12 renamed OUT_12
- net OUT_12: no longer J1.31 (Pin_31)
- net IN_13 renamed OUT_13
- net OUT_13: no longer J1.33 (Pin_33)
- net IN_14 renamed OUT_14
- net OUT_14: no longer J1.35 (Pin_35)
- net IN_15 renamed OUT_15
- net OUT_15: no longer J1.37 (Pin_37)
- net IN_2 renamed OUT_2
- net OUT_2: no longer J1.7 (Pin_7)
- net IN_3 renamed OUT_3
- net OUT_3: no longer J1.9 (Pin_9)
- net IN_4 renamed OUT_4
- net OUT_4: no longer J1.11 (Pin_11)
- net IN_5 renamed OUT_5
- net OUT_5: no longer J1.13 (Pin_13)
- net IN_6 renamed OUT_6
- net OUT_6: no longer J1.17 (Pin_17)
- net IN_7 renamed OUT_7
- net OUT_7: no longer J1.19 (Pin_19)
- net IN_8 renamed OUT_8
- net OUT_8: no longer J1.21 (Pin_21)
- net IN_9 renamed OUT_9
- net OUT_9: no longer J1.23 (Pin_23)
