File: KiCad/Serial Module/FPGA_Connector.kicad_sch (KiCad schematic)
At the start: 9 parts, among them J1 Conn_02x25_Odd_Even, U2 D1213A-04S-7, U3 D1213A-04S-7, U4 D1213A-04S-7, U5 D1213A-04S-7, U6 D1213A-04S-7

Commit message: Serial Module: review fixes, full BOM part numbers, stock footprints
Schematic fixes:
- +24V_PORT tied to +24V; STM32 VBAT tied to VDD
- Pull-ups on CONFIG15-18 and on bias-buffer OE inputs; pull-downs on PC13/PC14
- CONFIG_UPDATE moved from PC15 to PC7; VCXO Vcon biased to 1.65 V
- RJ45 LED anodes moved from 5V_LOGIC to 3.3V
- 74LVC125 units kept within one transceiver-pair instance; fixed pair-1
  annotation (U27/U28 units) that shorted MUX_B to DI_B in the netlist
- 5 V bias buffers changed to TI SN74ACT125PWR (TTL inputs, 4.5-5.5 V)
- Current-limit NMOS changed to AO3400A (Transistor_FET symbol, SOT-23 G/S/D)
- 24 V input TVS changed to TI TVS2700DRVR flat-clamp (27 V standoff,
  35 V max clamp at 40 A) replacing PTVS26VZ1USK (42 V clamp)
- Removed unused port_vsense_muc.kicad_sch

BOM and footprints:
- Every part now has Manufacturer, Part number and LCSC# (verified in stock);
  YAGEO caps/resistors, TI logic where stocked
- 24 V-rail MLCCs now 10 uF 50 V X7R 1210; bulk caps 100 uF 50 V
- TPS274160B footprint corrected to VQFN-28 4x5 mm (RLH); THVD1420 to
  150-mil SOIC-8; all custom footprints replaced with KiCad stock except
  J1 (card connector) and J3 (2x4 RJ45)
- "Part Number" fields normalised to "Part number"

Co-Authored-By: Claude Opus 5.5 <noreply@anthropic.com>
Parts:
- C13: value 22uf -> 10uF; footprint Capacitor_SMD:C_1206_3216Metric -> Capacitor_SMD:C_1210_3225Metric; LCSC# C12891 -> C596319; Manufacturer Samsung Electro-Mechanics -> YAGEO; Part number CL31A226KAHNNNE -> CC1210KKX7R9BB106; cost 0.04 -> 0.3958
- J1: Part Number X4621WR-2x25I-C40D28 -> (none); Part number (none) -> X4621WR-2x25I-C40D28
- U2, U3, U4, U5, U6: footprint footprints:SOT-363_DIO -> Package_TO_SOT_SMD:SOT-363_SC-70-6; Part Number D1213A-04S-7-ES -> (none); Part number (none) -> D1213A-04S-7-ES
