File: KiCad/Serial Module/Serial Module.kicad_pcb (KiCad board)
At the start: 4 copper layers, 75 x 100 mm, 46 parts, among them J1 Conn_02x25_Odd_Even, J2 Conn_ARM_SWD_TagConnect_TC2030, U1 STM32F411RETx, U2 D1213A-04S-7, U3 D1213A-04S-7, U4 D1213A-04S-7, U5 D1213A-04S-7, U6 D1213A-04S-7, U7 74LVC1G126, U8 74LVC1G126, X1 25Mhz

Commit message: update serial module and backplane hw
Parts:
- added C100: .1uf, Capacitor_SMD:C_0603_1608Metric, F.Cu at (353.1, 101.7)
- added C101: .1uf, Capacitor_SMD:C_0603_1608Metric, F.Cu at (357.1, 91.7)
- added C102: .1uf, Capacitor_SMD:C_0603_1608Metric, F.Cu at (357.1, 94.2)
- added C103: .1uf, Capacitor_SMD:C_0603_1608Metric, F.Cu at (357.1, 96.7)
- added C104: 22uf, Capacitor_SMD:C_1206_3216Metric, F.Cu at (357.1, 99.2)
- added C105: .1uf, Capacitor_SMD:C_0603_1608Metric, F.Cu at (357.1, 101.7)
- added C106: .1uf, Capacitor_SMD:C_0603_1608Metric, F.Cu at (361.1, 91.7)
- added C107: .1uf, Capacitor_SMD:C_0603_1608Metric, F.Cu at (361.1, 94.2)
- added C108: .1uf, Capacitor_SMD:C_0603_1608Metric, F.Cu at (361.1, 96.7)
- added C109: .1uf, Capacitor_SMD:C_0603_1608Metric, F.Cu at (361.1, 99.2)
- added C110: 22uf, Capacitor_SMD:C_1206_3216Metric, F.Cu at (289.3, 99.0)
- added C111: .1uf, Capacitor_SMD:C_0603_1608Metric, F.Cu at (278.5, 98.6)
- added C112: .1uf, Capacitor_SMD:C_0402_1005Metric, F.Cu at (296.5, 98.3)
- added C113: .1uf, Capacitor_SMD:C_0402_1005Metric, F.Cu at (296.5, 100.3)
- added C114: 75pf, Capacitor_SMD:C_0402_1005Metric, F.Cu at (296.5, 102.2)
- added C115: 22uf, Capacitor_SMD:C_1206_3216Metric, F.Cu at (289.3, 102.3)
- added C116: 22uf, Capacitor_SMD:C_1206_3216Metric, F.Cu at (289.3, 105.7)
- added C117: .1uf, Capacitor_SMD:C_0603_1608Metric, F.Cu at (251.3, 98.6)
- added C118: .1uf, Capacitor_SMD:C_0603_1608Metric, F.Cu at (251.3, 101.1)
- added C119: .1uf, Capacitor_SMD:C_0603_1608Metric, F.Cu at (251.3, 103.6)
- added C120: 22uf, Capacitor_SMD:C_1206_3216Metric, F.Cu at (251.3, 106.1)
- added C121: .1uf, Capacitor_SMD:C_0603_1608Metric, F.Cu at (251.3, 108.6)
- added C122: .1uf, Capacitor_SMD:C_0603_1608Metric, F.Cu at (251.3, 111.1)
- added C123: .1uf, Capacitor_SMD:C_0603_1608Metric, F.Cu at (251.3, 113.6)
- added C124: .1uf, Capacitor_SMD:C_0603_1608Metric, F.Cu at (260.4, 126.0)
- added C125: .1uf, Capacitor_SMD:C_0603_1608Metric, F.Cu at (260.4, 128.5)
- added C126: .1uf, Capacitor_SMD:C_0603_1608Metric, F.Cu at (260.4, 131.0)
- added C127: .1uf, Capacitor_SMD:C_0603_1608Metric, F.Cu at (260.4, 133.5)
- added C128: .1uf, Capacitor_SMD:C_0603_1608Metric, F.Cu at (260.4, 136.0)
- added C129: 22uf, Capacitor_SMD:C_1206_3216Metric, F.Cu at (260.4, 138.5)
- added C130: .1uf, Capacitor_SMD:C_0603_1608Metric, F.Cu at (264.4, 126.0)
- added C131: .1uf, Capacitor_SMD:C_0603_1608Metric, F.Cu at (264.4, 128.5)
- added C132: 22uf, Capacitor_SMD:C_1206_3216Metric, F.Cu at (304.8, 105.8)
- added C133: .1uf, Capacitor_SMD:C_0402_1005Metric, F.Cu at (318.0, 105.1)
- added C134: .1uf, Capacitor_SMD:C_0402_1005Metric, F.Cu at (318.0, 107.1)
- added C135: 75pf, Capacitor_SMD:C_0402_1005Metric, F.Cu at (318.0, 109.0)
- added C136: 22uf, Capacitor_SMD:C_1206_3216Metric, F.Cu at (304.8, 109.1)
- added C137: 22uf, Capacitor_SMD:C_1206_3216Metric, F.Cu at (304.8, 112.5)
- added C138: .1uf, Capacitor_SMD:C_0603_1608Metric, F.Cu at (309.6, 105.4)
- added C139: .1uf, Capacitor_SMD:C_0603_1608Metric, F.Cu at (309.6, 107.9)
- added C140: 22uf, Capacitor_SMD:C_1206_3216Metric, F.Cu at (405.8, 83.7)
- added C141: .1uf, Capacitor_SMD:C_0603_1608Metric, F.Cu at (393.4, 64.2)
- added C142: .1uf, Capacitor_SMD:C_0603_1608Metric, F.Cu at (393.4, 66.7)
- added C143: .1uf, Capacitor_SMD:C_0603_1608Metric, F.Cu at (393.4, 69.2)
- added C144: .1uf, Capacitor_SMD:C_0603_1608Metric, F.Cu at (393.4, 71.7)
- added C145: .1uf, Capacitor_SMD:C_0603_1608Metric, F.Cu at (393.4, 74.2)
- added C146: .1uf, Capacitor_SMD:C_0603_1608Metric, F.Cu at (393.4, 76.7)
- added C147: 22uf, Capacitor_SMD:C_1206_3216Metric, F.Cu at (398.2, 64.6)
- added C148: .1uf, Capacitor_SMD:C_0603_1608Metric, F.Cu at (416.2, 78.3)
- added C149: .1uf, Capacitor_SMD:C_0603_1608Metric, F.Cu at (405.0, 64.2)
- added C150: .1uf, Capacitor_SMD:C_0603_1608Metric, F.Cu at (405.0, 73.7)
- added C151: .1uf, Capacitor_SMD:C_0603_1608Metric, F.Cu at (405.0, 76.2)
- added C152: .1uf, Capacitor_SMD:C_0603_1608Metric, F.Cu at (405.0, 78.7)
- added C17: .1uf, Capacitor_SMD:C_0603_1608Metric, F.Cu at (213.6, 80.5)
- added C19: .1uf, Capacitor_SMD:C_0603_1608Metric, F.Cu at (213.6, 83.1)
- added C20: 22nf, Capacitor_SMD:C_0603_1608Metric, F.Cu at (335.0, 23.2)
- added C21: 22nf, Capacitor_SMD:C_0603_1608Metric, F.Cu at (335.0, 25.7)
- added C22: 22nf, Capacitor_SMD:C_0603_1608Metric, F.Cu at (335.0, 28.2)
- added C23: 22nf, Capacitor_SMD:C_0603_1608Metric, F.Cu at (335.0, 30.8)
- added C24: 22uf, Capacitor_SMD:C_1206_3216Metric, F.Cu at (355.8, 23.6)
- added C25: .1uf, Capacitor_SMD:C_0603_1608Metric, F.Cu at (209.0, 66.5)
- added C26: .1uf, Capacitor_SMD:C_0603_1608Metric, F.Cu at (209.0, 69.0)
- added C27: .1uf, Capacitor_SMD:C_0603_1608Metric, F.Cu at (335.0, 33.3)
- added C28: 22uf, Capacitor_SMD:C_1206_3216Metric, F.Cu at (355.8, 27.0)
- added C29: 120uf, Capacitor_SMD:CP_Elec_8x10.5, F.Cu at (326.3, 27.0)
- added C30: .1uf, Capacitor_SMD:C_0603_1608Metric, F.Cu at (335.0, 35.8)
- added C31: .1uf, Capacitor_SMD:C_0603_1608Metric, F.Cu at (384.1, 23.2)
- added C32: .1uf, Capacitor_SMD:C_0603_1608Metric, F.Cu at (384.1, 25.7)
- added C33: .1uf, Capacitor_SMD:C_0603_1608Metric, F.Cu at (335.0, 38.3)
- added C34: 120uf, Capacitor_SMD:CP_Elec_8x10.5, F.Cu at (326.3, 37.0)
- added C35: 22uf, Capacitor_SMD:C_1206_3216Metric, F.Cu at (355.8, 30.3)
- added C36: 22uf, Capacitor_SMD:C_1206_3216Metric, F.Cu at (355.8, 33.7)
- added C37: 22nf, Capacitor_SMD:C_0603_1608Metric, F.Cu at (335.0, 40.8)
- added C38: .1uf, Capacitor_SMD:C_0603_1608Metric, F.Cu at (335.0, 43.3)
- added C39: 22nf, Capacitor_SMD:C_0603_1608Metric, F.Cu at (335.0, 45.8)
- added C40: 22nf, Capacitor_SMD:C_0603_1608Metric, F.Cu at (335.0, 48.3)
- added C41: 22nf, Capacitor_SMD:C_0603_1608Metric, F.Cu at (339.0, 23.2)
- added C42: .1uf, Capacitor_SMD:C_0603_1608Metric, F.Cu at (339.0, 25.7)
- added C43: .1uf, Capacitor_SMD:C_0603_1608Metric, F.Cu at (339.0, 28.2)
- added C44: 120uf, Capacitor_SMD:CP_Elec_8x10.5, F.Cu at (326.3, 47.1)
- added C45: 120uf, Capacitor_SMD:CP_Elec_8x10.5, F.Cu at (326.3, 57.1)
- added C46: 22uf, Capacitor_SMD:C_1206_3216Metric, F.Cu at (355.8, 37.0)
- added C47: 22uf, Capacitor_SMD:C_1206_3216Metric, F.Cu at (355.8, 40.4)
- added C48: 22uf, Capacitor_SMD:C_1206_3216Metric, F.Cu at (355.8, 43.7)
- added C49: 22uf, Capacitor_SMD:C_1206_3216Metric, F.Cu at (355.8, 47.1)
- added C50: 22nf, Capacitor_SMD:C_0603_1608Metric, F.Cu at (339.0, 30.8)
- added C51: 22nf, Capacitor_SMD:C_0603_1608Metric, F.Cu at (339.0, 33.3)
- added C52: .1uf, Capacitor_SMD:C_0603_1608Metric, F.Cu at (339.0, 35.8)
- added C53: .1uf, Capacitor_SMD:C_0603_1608Metric, F.Cu at (339.0, 38.3)
- added C54: 22nf, Capacitor_SMD:C_0603_1608Metric, F.Cu at (339.0, 40.8)
- added C55: 22nf, Capacitor_SMD:C_0603_1608Metric, F.Cu at (339.0, 43.3)
- added C56: 22nf, Capacitor_SMD:C_0603_1608Metric, F.Cu at (339.0, 45.8)
- added C57: 22nf, Capacitor_SMD:C_0603_1608Metric, F.Cu at (339.0, 48.3)
- added C58: 22nf, Capacitor_SMD:C_0603_1608Metric, F.Cu at (343.0, 23.2)
- added C59: 22nf, Capacitor_SMD:C_0603_1608Metric, F.Cu at (343.0, 25.7)
- added C60: .1uf, Capacitor_SMD:C_0603_1608Metric, F.Cu at (343.0, 28.2)
- added C61: .1uf, Capacitor_SMD:C_0603_1608Metric, F.Cu at (343.0, 30.8)
- added C62: .1uf, Capacitor_SMD:C_0603_1608Metric, F.Cu at (343.0, 33.3)
- added C63: .1uf, Capacitor_SMD:C_0603_1608Metric, F.Cu at (343.0, 35.8)
- added C64: .1uf, Capacitor_SMD:C_0603_1608Metric, F.Cu at (343.0, 38.3)
- added C65: .1uf, Capacitor_SMD:C_0603_1608Metric, F.Cu at (343.0, 40.8)
- added C66: .1uf, Capacitor_SMD:C_0603_1608Metric, F.Cu at (343.0, 43.3)
- added C67: .1uf, Capacitor_SMD:C_0603_1608Metric, F.Cu at (343.0, 45.8)
- added C68: .1uf, Capacitor_SMD:C_0603_1608Metric, F.Cu at (287.4, 66.8)
- added C69: .1uf, Capacitor_SMD:C_0603_1608Metric, F.Cu at (287.4, 69.4)
- added C70: .1uf, Capacitor_SMD:C_0603_1608Metric, F.Cu at (287.4, 71.9)
- added C71: .1uf, Capacitor_SMD:C_0603_1608Metric, F.Cu at (287.4, 74.4)
- added C72: .1uf, Capacitor_SMD:C_0603_1608Metric, F.Cu at (287.4, 21.5)
- added C73: .1uf, Capacitor_SMD:C_0603_1608Metric, F.Cu at (287.4, 24.0)
- added C74: .1uf, Capacitor_SMD:C_0603_1608Metric, F.Cu at (287.4, 26.5)
- added C75: .1uf, Capacitor_SMD:C_0603_1608Metric, F.Cu at (287.4, 29.0)
- added C76: 22uf, Capacitor_SMD:C_1206_3216Metric, F.Cu at (265.9, 44.2)
- added C77: .1uf, Capacitor_SMD:C_0603_1608Metric, F.Cu at (265.9, 46.7)
- added C78: .1uf, Capacitor_SMD:C_0603_1608Metric, F.Cu at (265.9, 49.2)
- added C79: .1uf, Capacitor_SMD:C_0603_1608Metric, F.Cu at (265.9, 51.7)
- added C80: .1uf, Capacitor_SMD:C_0603_1608Metric, F.Cu at (244.5, 44.2)
- added C81: .1uf, Capacitor_SMD:C_0603_1608Metric, F.Cu at (244.5, 46.7)
- added C82: .1uf, Capacitor_SMD:C_0603_1608Metric, F.Cu at (244.5, 49.2)
- added C83: .1uf, Capacitor_SMD:C_0603_1608Metric, F.Cu at (244.5, 51.7)
- added C84: .1uf, Capacitor_SMD:C_0603_1608Metric, F.Cu at (287.4, 44.2)
- added C85: 22uf, Capacitor_SMD:C_1206_3216Metric, F.Cu at (287.4, 46.7)
- added C86: .1uf, Capacitor_SMD:C_0603_1608Metric, F.Cu at (287.4, 49.2)
- added C87: .1uf, Capacitor_SMD:C_0603_1608Metric, F.Cu at (287.4, 51.7)
- added C88: .1uf, Capacitor_SMD:C_0603_1608Metric, F.Cu at (265.9, 21.5)
- added C89: .1uf, Capacitor_SMD:C_0603_1608Metric, F.Cu at (265.9, 24.0)
- added C90: .1uf, Capacitor_SMD:C_0603_1608Metric, F.Cu at (265.9, 26.5)
- added C91: .1uf, Capacitor_SMD:C_0603_1608Metric, F.Cu at (265.9, 29.0)
- added C92: .1uf, Capacitor_SMD:C_0603_1608Metric, F.Cu at (244.5, 21.5)
- added C93: .1uf, Capacitor_SMD:C_0603_1608Metric, F.Cu at (244.5, 24.0)
- added C94: 22uf, Capacitor_SMD:C_1206_3216Metric, F.Cu at (244.5, 26.5)
- added C95: .1uf, Capacitor_SMD:C_0603_1608Metric, F.Cu at (244.5, 29.0)
- added C96: .1uf, Capacitor_SMD:C_0603_1608Metric, F.Cu at (353.1, 91.7)
- added C97: .1uf, Capacitor_SMD:C_0603_1608Metric, F.Cu at (353.1, 94.2)
- added C98: .1uf, Capacitor_SMD:C_0603_1608Metric, F.Cu at (353.1, 96.7)
- added C99: .1uf, Capacitor_SMD:C_0603_1608Metric, F.Cu at (353.1, 99.2)
- added D10: D_Schottky, Diode_SMD:D_SOD-123F, F.Cu at (337.0, 61.0)
- added D11: D_Schottky, Diode_SMD:D_SOD-123F, F.Cu at (337.0, 65.5)
- added D12: D_Schottky, Diode_SMD:D_SOD-123F, F.Cu at (337.0, 70.0)
- added D13: D_Schottky, Diode_SMD:D_SOD-123F, F.Cu at (345.1, 51.9)
- added D14: D_Schottky, Diode_SMD:D_SOD-123F, F.Cu at (345.1, 56.4)
- added D15: D_Schottky, Diode_SMD:D_SOD-123F, F.Cu at (345.1, 61.0)
- added D16: D_Schottky, Diode_SMD:D_SOD-123F, F.Cu at (345.1, 65.5)
- added D17: D_Schottky, Diode_SMD:D_SOD-123F, F.Cu at (345.1, 70.0)
- added D18: D_Schottky, Diode_SMD:D_SOD-123F, F.Cu at (353.2, 51.9)
- added D19: D_Schottky, Diode_SMD:D_SOD-123F, F.Cu at (353.2, 56.4)
- added D20: D_Schottky, Diode_SMD:D_SOD-123F, F.Cu at (353.2, 61.0)
- added D21: D_Schottky, Diode_SMD:D_SOD-123F, F.Cu at (353.2, 65.5)
- added D22: D_Schottky, Diode_SMD:D_SOD-123F, F.Cu at (353.2, 70.0)
- added D23: D_Schottky, Diode_SMD:D_SOD-123F, F.Cu at (361.3, 51.9)
- added D24: D_Schottky, Diode_SMD:D_SOD-123F, F.Cu at (361.3, 56.4)
- added D25: D_Schottky, Diode_SMD:D_SOD-123F, F.Cu at (361.3, 61.0)
- added D26: D_Schottky, Diode_SMD:D_SOD-123F, F.Cu at (361.3, 65.5)
- added D27: D_Schottky, Diode_SMD:D_SOD-123F, F.Cu at (361.3, 70.0)
- added D28: BAT54SLT1G, Package_TO_SOT_SMD:SOT-23, F.Cu at (353.8, 74.5)
- added D29: BAT54SLT1G, Package_TO_SOT_SMD:SOT-23, F.Cu at (353.8, 79.0)
- added D30: BAT54SLT1G, Package_TO_SOT_SMD:SOT-23, F.Cu at (358.7, 74.5)
- added D31: BAT54SLT1G, Package_TO_SOT_SMD:SOT-23, F.Cu at (358.7, 79.0)
- added D32: BAT54SLT1G, Package_TO_SOT_SMD:SOT-23, F.Cu at (363.6, 74.5)
- added D33: BAT54SLT1G, Package_TO_SOT_SMD:SOT-23, F.Cu at (363.6, 79.0)
- added D34: BAT54SLT1G, Package_TO_SOT_SMD:SOT-23, F.Cu at (368.5, 74.5)
- added D35: BAT54SLT1G, Package_TO_SOT_SMD:SOT-23, F.Cu at (368.5, 79.0)
- added D36: SM712_SOT23, Package_TO_SOT_SMD:SOT-23, F.Cu at (299.8, 67.8)
- added D37: SM712_SOT23, Package_TO_SOT_SMD:SOT-23, F.Cu at (299.8, 72.3)
- added D38: SM712_SOT23, Package_TO_SOT_SMD:SOT-23, F.Cu at (299.8, 22.4)
- added D39: SM712_SOT23, Package_TO_SOT_SMD:SOT-23, F.Cu at (299.8, 26.9)
- added D40: SM712_SOT23, Package_TO_SOT_SMD:SOT-23, F.Cu at (278.4, 45.1)
- added D41: SM712_SOT23, Package_TO_SOT_SMD:SOT-23, F.Cu at (278.4, 49.6)
- added D42: SM712_SOT23, Package_TO_SOT_SMD:SOT-23, F.Cu at (257.0, 45.1)
- added D43: SM712_SOT23, Package_TO_SOT_SMD:SOT-23, F.Cu at (257.0, 49.6)
- added D44: SM712_SOT23, Package_TO_SOT_SMD:SOT-23, F.Cu at (299.8, 45.1)
- added D45: SM712_SOT23, Package_TO_SOT_SMD:SOT-23, F.Cu at (299.8, 49.6)
- added D46: SM712_SOT23, Package_TO_SOT_SMD:SOT-23, F.Cu at (278.4, 22.4)
- added D47: SM712_SOT23, Package_TO_SOT_SMD:SOT-23, F.Cu at (278.4, 26.9)
- added D48: SM712_SOT23, Package_TO_SOT_SMD:SOT-23, F.Cu at (257.0, 22.4)
- added D49: SM712_SOT23, Package_TO_SOT_SMD:SOT-23, F.Cu at (257.0, 26.9)
- added D50: BAT54SLT1G, Package_TO_SOT_SMD:SOT-23, F.Cu at (314.1, 106.3)
- added D51: BAT54SLT1G, Package_TO_SOT_SMD:SOT-23, F.Cu at (314.1, 110.8)
- added D6: SM712_SOT23, Package_TO_SOT_SMD:SOT-23, F.Cu at (230.9, 71.2)
- added D7: SM712_SOT23, Package_TO_SOT_SMD:SOT-23, F.Cu at (230.9, 75.6)
- added D8: D_Schottky, Diode_SMD:D_SOD-123F, F.Cu at (337.0, 51.9)
- added D9: D_Schottky, Diode_SMD:D_SOD-123F, F.Cu at (337.0, 56.4)
- added J3: ~, footprints:RJ45-TH_HC-RJ45-059D-2X4-2-04, F.Cu at (161.6, 85.5)
- added JP1: Jumper_3_Bridged12, Connector_PinHeader_2.54mm:PinHeader_1x03_P2.54mm_Vertical, F.Cu at (335.2, 74.6)
- added JP2: Jumper_3_Bridged12, Connector_PinHeader_2.54mm:PinHeader_1x03_P2.54mm_Vertical, F.Cu at (339.8, 74.6)
- added JP3: Jumper_3_Bridged12, Connector_PinHeader_2.54mm:PinHeader_1x03_P2.54mm_Vertical, F.Cu at (344.4, 74.6)
- added JP4: Jumper_3_Bridged12, Connector_PinHeader_2.54mm:PinHeader_1x03_P2.54mm_Vertical, F.Cu at (349.0, 74.6)
- added L1: 15uH, footprints:FCH0650, F.Cu at (306.9, 99.9)
- added L5: 15uH, footprints:FCH0650, F.Cu at (295.8, 108.7)
- added R10: 10K, Resistor_SMD:R_0603_1608Metric, F.Cu at (213.6, 85.6)
- added R100: 470, Resistor_SMD:R_0603_1608Metric, F.Cu at (277.4, 58.6)
- added R101: 10K, Resistor_SMD:R_0603_1608Metric, F.Cu at (274.0, 49.2)
- added R102: 10K, Resistor_SMD:R_0603_1608Metric, F.Cu at (274.0, 51.7)
- added R103: 10, Resistor_SMD:R_0603_1608Metric, F.Cu at (244.5, 54.2)
- added R104: 10, Resistor_SMD:R_0603_1608Metric, F.Cu at (244.5, 56.7)
- added R105: 10, Resistor_SMD:R_0402_1005Metric, F.Cu at (248.5, 44.2)
- added R106: 10, Resistor_SMD:R_0402_1005Metric, F.Cu at (248.5, 46.7)
- added R107: 137, Resistor_SMD:R_0603_1608Metric, F.Cu at (248.5, 49.2)
- added R108: 137, Resistor_SMD:R_0603_1608Metric, F.Cu at (248.5, 51.7)
- added R109: 10K, Resistor_SMD:R_0603_1608Metric, F.Cu at (248.5, 54.2)
- added R11: 10K, Resistor_SMD:R_0603_1608Metric, F.Cu at (213.6, 88.1)
- added R110: 10K, Resistor_SMD:R_0603_1608Metric, F.Cu at (248.5, 56.7)
- added R111: 10K, Resistor_SMD:R_0603_1608Metric, F.Cu at (252.6, 44.2)
- added R112: 10K, Resistor_SMD:R_0603_1608Metric, F.Cu at (252.6, 46.7)
- added R113: 10K, Resistor_SMD:R_0603_1608Metric, F.Cu at (256.0, 56.6)
- added R114: 10K, Resistor_SMD:R_0603_1608Metric, F.Cu at (256.0, 58.6)
- added R115: 10K, Resistor_SMD:R_0603_1608Metric, F.Cu at (252.6, 49.2)
- added R116: 10K, Resistor_SMD:R_0603_1608Metric, F.Cu at (252.6, 51.7)
- added R117: 10K, Resistor_SMD:R_0603_1608Metric, F.Cu at (287.4, 54.2)
- added R118: 10K, Resistor_SMD:R_0603_1608Metric, F.Cu at (287.4, 56.7)
- added R119: 10K, Resistor_SMD:R_0603_1608Metric, F.Cu at (291.4, 44.2)
- added R12: 10K, Resistor_SMD:R_0603_1608Metric, F.Cu at (213.6, 90.6)
- added R120: 10K, Resistor_SMD:R_0603_1608Metric, F.Cu at (291.4, 46.7)
- added R121: 470, Resistor_SMD:R_0603_1608Metric, F.Cu at (291.4, 49.2)
- added R122: 470, Resistor_SMD:R_0603_1608Metric, F.Cu at (291.4, 51.7)
- added R123: 470, Resistor_SMD:R_0603_1608Metric, F.Cu at (291.4, 54.2)
- added R124: 470, Resistor_SMD:R_0603_1608Metric, F.Cu at (291.4, 56.7)
- added R125: 10K, Resistor_SMD:R_0603_1608Metric, F.Cu at (295.4, 44.2)
- added R126: 10K, Resistor_SMD:R_0603_1608Metric, F.Cu at (295.4, 46.7)
- added R127: 10, Resistor_SMD:R_0603_1608Metric, F.Cu at (298.8, 56.6)
- added R128: 10, Resistor_SMD:R_0603_1608Metric, F.Cu at (298.8, 58.6)
- added R129: 10, Resistor_SMD:R_0402_1005Metric, F.Cu at (295.4, 49.2)
- added R13: 10K, Resistor_SMD:R_0603_1608Metric, F.Cu at (217.6, 80.5)
- added R130: 10, Resistor_SMD:R_0402_1005Metric, F.Cu at (295.4, 51.7)
- added R131: 137, Resistor_SMD:R_0603_1608Metric, F.Cu at (265.9, 31.5)
- added R132: 137, Resistor_SMD:R_0603_1608Metric, F.Cu at (265.9, 34.0)
- added R133: 10K, Resistor_SMD:R_0603_1608Metric, F.Cu at (269.9, 21.5)
- added R134: 10K, Resistor_SMD:R_0603_1608Metric, F.Cu at (269.9, 24.0)
- added R135: 10K, Resistor_SMD:R_0603_1608Metric, F.Cu at (269.9, 26.5)
- added R136: 10K, Resistor_SMD:R_0603_1608Metric, F.Cu at (269.9, 29.0)
- added R137: 10K, Resistor_SMD:R_0603_1608Metric, F.Cu at (269.9, 31.5)
- added R138: 10K, Resistor_SMD:R_0603_1608Metric, F.Cu at (269.9, 34.0)
- added R139: 10K, Resistor_SMD:R_0603_1608Metric, F.Cu at (274.0, 21.5)
- added R14: 470, Resistor_SMD:R_0603_1608Metric, F.Cu at (217.6, 83.1)
- added R140: 10K, Resistor_SMD:R_0603_1608Metric, F.Cu at (274.0, 24.0)
- added R141: 10K, Resistor_SMD:R_0603_1608Metric, F.Cu at (277.4, 33.9)
- added R142: 10K, Resistor_SMD:R_0603_1608Metric, F.Cu at (277.4, 35.9)
- added R143: 10K, Resistor_SMD:R_0603_1608Metric, F.Cu at (274.0, 26.5)
- added R144: 10K, Resistor_SMD:R_0603_1608Metric, F.Cu at (274.0, 29.0)
- added R145: 470, Resistor_SMD:R_0603_1608Metric, F.Cu at (244.5, 31.5)
- added R146: 470, Resistor_SMD:R_0603_1608Metric, F.Cu at (244.5, 34.0)
- added R147: 470, Resistor_SMD:R_0603_1608Metric, F.Cu at (248.5, 21.5)
- added R148: 470, Resistor_SMD:R_0603_1608Metric, F.Cu at (248.5, 24.0)
- added R149: 10K, Resistor_SMD:R_0603_1608Metric, F.Cu at (248.5, 26.5)
- added R15: 470, Resistor_SMD:R_0603_1608Metric, F.Cu at (217.6, 85.6)
- added R150: 10K, Resistor_SMD:R_0603_1608Metric, F.Cu at (248.5, 29.0)
- added R151: 10, Resistor_SMD:R_0603_1608Metric, F.Cu at (248.5, 31.5)
- added R152: 10, Resistor_SMD:R_0603_1608Metric, F.Cu at (248.5, 34.0)
- added R153: 10, Resistor_SMD:R_0402_1005Metric, F.Cu at (252.6, 21.5)
- added R154: 10, Resistor_SMD:R_0402_1005Metric, F.Cu at (252.6, 24.0)
- added R155: 137, Resistor_SMD:R_0603_1608Metric, F.Cu at (256.0, 33.9)
- added R156: 137, Resistor_SMD:R_0603_1608Metric, F.Cu at (256.0, 35.9)
- added R157: 10K, Resistor_SMD:R_0603_1608Metric, F.Cu at (252.6, 26.5)
- added R158: 10K, Resistor_SMD:R_0603_1608Metric, F.Cu at (252.6, 29.0)
- added R159: 10K, Resistor_SMD:R_0603_1608Metric, F.Cu at (278.5, 101.1)
- added R16: 470, Resistor_SMD:R_0603_1608Metric, F.Cu at (217.6, 88.1)
- added R160: 10k, Resistor_SMD:R_0603_1608Metric, F.Cu at (293.6, 98.3)
- added R161: 10k, Resistor_SMD:R_0603_1608Metric, F.Cu at (293.6, 100.3)
- added R162: 100k, Resistor_SMD:R_0402_1005Metric, F.Cu at (293.6, 102.3)
- added R163: 12.4k, Resistor_SMD:R_0402_1005Metric, F.Cu at (293.6, 104.3)
- added R164: 10K, Resistor_SMD:R_0603_1608Metric, F.Cu at (282.5, 126.0)
- added R165: 10K, Resistor_SMD:R_0603_1608Metric, F.Cu at (282.5, 128.5)
- added R166: 10K, Resistor_SMD:R_0603_1608Metric, F.Cu at (282.5, 131.0)
- added R167: 10K, Resistor_SMD:R_0603_1608Metric, F.Cu at (282.5, 133.5)
- added R168: 10K, Resistor_SMD:R_0603_1608Metric, F.Cu at (282.5, 136.0)
- added R169: 10K, Resistor_SMD:R_0603_1608Metric, F.Cu at (286.5, 126.0)
- added R17: 470, Resistor_SMD:R_0603_1608Metric, F.Cu at (217.6, 90.6)
- added R170: 10K, Resistor_SMD:R_0603_1608Metric, F.Cu at (286.5, 128.5)
- added R171: 10K, Resistor_SMD:R_0603_1608Metric, F.Cu at (278.5, 103.6)
- added R172: 10K, Resistor_SMD:R_0603_1608Metric, F.Cu at (286.5, 131.0)
- added R173: 10K, Resistor_SMD:R_0603_1608Metric, F.Cu at (286.5, 133.5)
- added R174: 10K, Resistor_SMD:R_0603_1608Metric, F.Cu at (286.5, 136.0)
- added R175: 470, Resistor_SMD:R_0603_1608Metric, F.Cu at (290.5, 126.0)
- added R176: 470, Resistor_SMD:R_0603_1608Metric, F.Cu at (290.5, 128.5)
- added R177: 470, Resistor_SMD:R_0603_1608Metric, F.Cu at (290.5, 131.0)
- added R178: 470, Resistor_SMD:R_0603_1608Metric, F.Cu at (290.5, 133.5)
- added R179: 10K, Resistor_SMD:R_0603_1608Metric, F.Cu at (278.5, 106.1)
- added R18: 10, Resistor_SMD:R_0603_1608Metric, F.Cu at (221.6, 80.5)
- added R180: 10K, Resistor_SMD:R_0603_1608Metric, F.Cu at (290.5, 136.0)
- added R181: 10K, Resistor_SMD:R_0603_1608Metric, F.Cu at (294.5, 126.0)
- added R182: 10, Resistor_SMD:R_0603_1608Metric, F.Cu at (294.5, 128.5)
- added R183: 10, Resistor_SMD:R_0603_1608Metric, F.Cu at (294.5, 131.0)
- added R184: 10, Resistor_SMD:R_0402_1005Metric, F.Cu at (281.9, 138.2)
- added R185: 10, Resistor_SMD:R_0402_1005Metric, F.Cu at (281.9, 140.2)
- added R186: 137, Resistor_SMD:R_0603_1608Metric, F.Cu at (294.5, 133.5)
- added R187: 10K, Resistor_SMD:R_0603_1608Metric, F.Cu at (278.5, 108.6)
- added R188: 137, Resistor_SMD:R_0603_1608Metric, F.Cu at (294.5, 136.0)
- added R189: 10K, Resistor_SMD:R_0603_1608Metric, F.Cu at (251.3, 116.1)
- added R19: 10, Resistor_SMD:R_0603_1608Metric, F.Cu at (221.6, 83.1)
- added R190: 10K, Resistor_SMD:R_0603_1608Metric, F.Cu at (255.3, 98.6)
- added R191: 10K, Resistor_SMD:R_0603_1608Metric, F.Cu at (255.3, 101.1)
- added R192: 10K, Resistor_SMD:R_0603_1608Metric, F.Cu at (255.3, 103.6)
- added R193: 10K, Resistor_SMD:R_0603_1608Metric, F.Cu at (255.3, 106.1)
- added R194: 10K, Resistor_SMD:R_0603_1608Metric, F.Cu at (255.3, 108.6)
- added R195: 10K, Resistor_SMD:R_0603_1608Metric, F.Cu at (278.5, 111.1)
- added R196: 10K, Resistor_SMD:R_0603_1608Metric, F.Cu at (255.3, 111.1)
- added R197: 10K, Resistor_SMD:R_0603_1608Metric, F.Cu at (255.3, 113.6)
- added R198: 10K, Resistor_SMD:R_0603_1608Metric, F.Cu at (255.3, 116.1)
- added R199: 10K, Resistor_SMD:R_0603_1608Metric, F.Cu at (259.3, 98.6)
- added R20: 10, Resistor_SMD:R_0402_1005Metric, F.Cu at (225.1, 84.1)
- added R200: 10K, Resistor_SMD:R_0603_1608Metric, F.Cu at (259.3, 101.1)
- added R201: 10K, Resistor_SMD:R_0603_1608Metric, F.Cu at (259.3, 103.6)
- added R202: 470, Resistor_SMD:R_0603_1608Metric, F.Cu at (259.3, 106.1)
- added R203: 10K, Resistor_SMD:R_0603_1608Metric, F.Cu at (282.5, 98.6)
- added R204: 470, Resistor_SMD:R_0603_1608Metric, F.Cu at (259.3, 108.6)
- added R205: 470, Resistor_SMD:R_0603_1608Metric, F.Cu at (259.3, 111.1)
- added R206: 470, Resistor_SMD:R_0603_1608Metric, F.Cu at (259.3, 113.6)
- added R207: 10K, Resistor_SMD:R_0603_1608Metric, F.Cu at (259.3, 116.1)
- added R208: 10K, Resistor_SMD:R_0603_1608Metric, F.Cu at (263.3, 98.6)
- added R209: 10, Resistor_SMD:R_0603_1608Metric, F.Cu at (263.3, 101.1)
- added R21: 10, Resistor_SMD:R_0402_1005Metric, F.Cu at (225.1, 86.1)
- added R210: 10, Resistor_SMD:R_0603_1608Metric, F.Cu at (263.3, 103.6)
- added R211: 10K, Resistor_SMD:R_0603_1608Metric, F.Cu at (282.5, 101.1)
- added R212: 10, Resistor_SMD:R_0402_1005Metric, F.Cu at (271.5, 118.1)
- added R213: 10, Resistor_SMD:R_0402_1005Metric, F.Cu at (271.5, 120.1)
- added R214: 137, Resistor_SMD:R_0603_1608Metric, F.Cu at (263.3, 106.1)
- added R215: 137, Resistor_SMD:R_0603_1608Metric, F.Cu at (263.3, 108.6)
- added R216: 10K, Resistor_SMD:R_0603_1608Metric, F.Cu at (264.4, 131.0)
- added R217: 10K, Resistor_SMD:R_0603_1608Metric, F.Cu at (264.4, 133.5)
- added R218: 10K, Resistor_SMD:R_0603_1608Metric, F.Cu at (264.4, 136.0)
- added R219: 10K, Resistor_SMD:R_0603_1608Metric, F.Cu at (282.5, 103.6)
- added R22: 137, Resistor_SMD:R_0603_1608Metric, F.Cu at (221.6, 85.6)
- added R220: 10K, Resistor_SMD:R_0603_1608Metric, F.Cu at (264.4, 138.5)
- added R221: 10K, Resistor_SMD:R_0603_1608Metric, F.Cu at (268.4, 126.0)
- added R222: 10K, Resistor_SMD:R_0603_1608Metric, F.Cu at (268.4, 128.5)
- added R223: 10K, Resistor_SMD:R_0603_1608Metric, F.Cu at (268.4, 131.0)
- added R224: 10K, Resistor_SMD:R_0603_1608Metric, F.Cu at (268.4, 133.5)
- added R225: 10K, Resistor_SMD:R_0603_1608Metric, F.Cu at (268.4, 136.0)
- added R226: 10K, Resistor_SMD:R_0603_1608Metric, F.Cu at (268.4, 138.5)
- added R227: 10K, Resistor_SMD:R_0603_1608Metric, F.Cu at (282.5, 106.1)
- added R228: 10K, Resistor_SMD:R_0603_1608Metric, F.Cu at (272.4, 126.0)
- added R229: 10K, Resistor_SMD:R_0603_1608Metric, F.Cu at (272.4, 128.5)
- added R23: 137, Resistor_SMD:R_0603_1608Metric, F.Cu at (221.6, 88.1)
- added R230: 470, Resistor_SMD:R_0603_1608Metric, F.Cu at (272.4, 131.0)
- added R231: 470, Resistor_SMD:R_0603_1608Metric, F.Cu at (272.4, 133.5)
- added R232: 470, Resistor_SMD:R_0603_1608Metric, F.Cu at (272.4, 136.0)
- added R233: 470, Resistor_SMD:R_0603_1608Metric, F.Cu at (272.4, 138.5)
- added R234: 10K, Resistor_SMD:R_0603_1608Metric, F.Cu at (276.5, 126.0)
- added R235: 10K, Resistor_SMD:R_0603_1608Metric, F.Cu at (282.5, 108.6)
- added R236: 10K, Resistor_SMD:R_0603_1608Metric, F.Cu at (276.5, 128.5)
- added R237: 10, Resistor_SMD:R_0603_1608Metric, F.Cu at (276.5, 131.0)
- added R238: 10, Resistor_SMD:R_0603_1608Metric, F.Cu at (276.5, 133.5)
- added R239: 10, Resistor_SMD:R_0402_1005Metric, F.Cu at (269.4, 140.8)
- added R24: 10k, Resistor_SMD:R_0603_1608Metric, F.Cu at (343.0, 48.3)
- added R240: 10, Resistor_SMD:R_0402_1005Metric, F.Cu at (269.4, 142.8)
- added R241: 137, Resistor_SMD:R_0603_1608Metric, F.Cu at (276.5, 136.0)
- added R242: 137, Resistor_SMD:R_0603_1608Metric, F.Cu at (276.5, 138.5)
- added R243: 10k, Resistor_SMD:R_0603_1608Metric, F.Cu at (309.6, 110.4)
- added R244: 10k, Resistor_SMD:R_0603_1608Metric, F.Cu at (309.6, 112.9)
- added R245: 100k, Resistor_SMD:R_0402_1005Metric, F.Cu at (318.0, 111.0)
- added R246: 13.3k, Resistor_SMD:R_0402_1005Metric, F.Cu at (318.0, 113.0)
- added R247: 10k, Resistor_SMD:R_0603_1608Metric, F.Cu at (405.0, 66.7)
- added R248: 10k, Resistor_SMD:R_0603_1608Metric, F.Cu at (405.0, 69.2)
- added R25: 10k, Resistor_SMD:R_0603_1608Metric, F.Cu at (347.0, 23.2)
- added R26: 10k, Resistor_SMD:R_0603_1608Metric, F.Cu at (347.0, 25.7)
- added R27: 10k, Resistor_SMD:R_0603_1608Metric, F.Cu at (347.0, 28.2)
- added R28: 10k, Resistor_SMD:R_0603_1608Metric, F.Cu at (347.0, 30.8)
- added R29: 10k, Resistor_SMD:R_0603_1608Metric, F.Cu at (347.0, 33.3)
- added R30: 1k, Resistor_SMD:R_0603_1608Metric, F.Cu at (347.0, 35.8)
- added R31: 10k, Resistor_SMD:R_0603_1608Metric, F.Cu at (347.0, 38.3)
- added R32: 1k, Resistor_SMD:R_0603_1608Metric, F.Cu at (347.0, 40.8)
- added R33: 10k, Resistor_SMD:R_0603_1608Metric, F.Cu at (347.0, 43.3)
- added R34: 1k, Resistor_SMD:R_0603_1608Metric, F.Cu at (347.0, 45.8)
- added R35: 10k, Resistor_SMD:R_0603_1608Metric, F.Cu at (347.0, 48.3)
- added R36: 1k, Resistor_SMD:R_0603_1608Metric, F.Cu at (351.0, 23.2)
- added R37: 10k, Resistor_SMD:R_0603_1608Metric, F.Cu at (351.0, 25.7)
- added R38: 1k, Resistor_SMD:R_0603_1608Metric, F.Cu at (351.0, 28.2)
- added R39: 10k, Resistor_SMD:R_0603_1608Metric, F.Cu at (351.0, 30.8)
- added R40: 1k, Resistor_SMD:R_0603_1608Metric, F.Cu at (351.0, 33.3)
- added R41: 10k, Resistor_SMD:R_0603_1608Metric, F.Cu at (351.0, 35.8)
- added R42: 1k, Resistor_SMD:R_0603_1608Metric, F.Cu at (351.0, 38.3)
- added R43: 10k, Resistor_SMD:R_0603_1608Metric, F.Cu at (351.0, 40.8)
- added R44: 1k, Resistor_SMD:R_0603_1608Metric, F.Cu at (351.0, 43.3)
- added R45: 1k, Resistor_SMD:R_0603_1608Metric, F.Cu at (265.9, 66.8)
- added R46: 1k, Resistor_SMD:R_0603_1608Metric, F.Cu at (265.9, 69.4)
- added R47: 1k, Resistor_SMD:R_0603_1608Metric, F.Cu at (265.9, 71.9)
- added R48: 1k, Resistor_SMD:R_0603_1608Metric, F.Cu at (265.9, 74.4)
- added R49: 1k, Resistor_SMD:R_0603_1608Metric, F.Cu at (265.9, 76.9)
- added R50: 1k, Resistor_SMD:R_0603_1608Metric, F.Cu at (265.9, 79.4)
- added R51: 1k, Resistor_SMD:R_0603_1608Metric, F.Cu at (269.9, 66.8)
- added R52: 1k, Resistor_SMD:R_0603_1608Metric, F.Cu at (269.9, 69.4)
- added R53: 1k, Resistor_SMD:R_0603_1608Metric, F.Cu at (269.9, 71.9)
- added R54: 1k, Resistor_SMD:R_0603_1608Metric, F.Cu at (269.9, 74.4)
- added R55: 1k, Resistor_SMD:R_0603_1608Metric, F.Cu at (269.9, 76.9)
- added R56: 1k, Resistor_SMD:R_0603_1608Metric, F.Cu at (269.9, 79.4)
- added R57: 1k, Resistor_SMD:R_0603_1608Metric, F.Cu at (274.0, 66.8)
- added R58: 1k, Resistor_SMD:R_0603_1608Metric, F.Cu at (274.0, 69.4)
- added R59: 1k, Resistor_SMD:R_0603_1608Metric, F.Cu at (274.0, 71.9)
- added R60: 1k, Resistor_SMD:R_0603_1608Metric, F.Cu at (274.0, 74.4)
- added R61: 10K, Resistor_SMD:R_0603_1608Metric, F.Cu at (287.4, 76.9)
- added R62: 10K, Resistor_SMD:R_0603_1608Metric, F.Cu at (287.4, 79.4)
- added R63: 10K, Resistor_SMD:R_0603_1608Metric, F.Cu at (291.4, 66.8)
- added R64: 10K, Resistor_SMD:R_0603_1608Metric, F.Cu at (291.4, 69.4)
- added R65: 10K, Resistor_SMD:R_0603_1608Metric, F.Cu at (291.4, 71.9)
- added R66: 10K, Resistor_SMD:R_0603_1608Metric, F.Cu at (291.4, 74.4)
- added R67: 10K, Resistor_SMD:R_0603_1608Metric, F.Cu at (291.4, 76.9)
- added R68: 10K, Resistor_SMD:R_0603_1608Metric, F.Cu at (291.4, 79.4)
- added R69: 10K, Resistor_SMD:R_0603_1608Metric, F.Cu at (295.4, 66.8)
- added R70: 10K, Resistor_SMD:R_0603_1608Metric, F.Cu at (295.4, 69.4)
- added R71: 10K, Resistor_SMD:R_0603_1608Metric, F.Cu at (298.8, 81.1)
- added R72: 10K, Resistor_SMD:R_0603_1608Metric, F.Cu at (298.8, 83.1)
- added R73: 470, Resistor_SMD:R_0603_1608Metric, F.Cu at (295.4, 71.9)
- added R74: 470, Resistor_SMD:R_0603_1608Metric, F.Cu at (295.4, 74.4)
- added R75: 470, Resistor_SMD:R_0603_1608Metric, F.Cu at (287.4, 31.5)
- added R76: 470, Resistor_SMD:R_0603_1608Metric, F.Cu at (287.4, 34.0)
- added R77: 10K, Resistor_SMD:R_0603_1608Metric, F.Cu at (291.4, 21.5)
- added R78: 10K, Resistor_SMD:R_0603_1608Metric, F.Cu at (291.4, 24.0)
- added R79: 10, Resistor_SMD:R_0603_1608Metric, F.Cu at (291.4, 26.5)
- added R80: 10, Resistor_SMD:R_0603_1608Metric, F.Cu at (291.4, 29.0)
- added R81: 10, Resistor_SMD:R_0402_1005Metric, F.Cu at (291.4, 31.5)
- added R82: 10, Resistor_SMD:R_0402_1005Metric, F.Cu at (291.4, 34.0)
- added R83: 137, Resistor_SMD:R_0603_1608Metric, F.Cu at (295.4, 21.5)
- added R84: 137, Resistor_SMD:R_0603_1608Metric, F.Cu at (295.4, 24.0)
- added R85: 10K, Resistor_SMD:R_0603_1608Metric, F.Cu at (298.8, 33.9)
- added R86: 10K, Resistor_SMD:R_0603_1608Metric, F.Cu at (298.8, 35.9)
- added R87: 10K, Resistor_SMD:R_0603_1608Metric, F.Cu at (295.4, 26.5)
- added R88: 10K, Resistor_SMD:R_0603_1608Metric, F.Cu at (295.4, 29.0)
- added R89: 10K, Resistor_SMD:R_0603_1608Metric, F.Cu at (265.9, 54.2)
- added R90: 10K, Resistor_SMD:R_0603_1608Metric, F.Cu at (265.9, 56.7)
- added R91: 10K, Resistor_SMD:R_0603_1608Metric, F.Cu at (269.9, 44.2)
- added R92: 10K, Resistor_SMD:R_0603_1608Metric, F.Cu at (269.9, 46.7)
- added R93: 10K, Resistor_SMD:R_0603_1608Metric, F.Cu at (269.9, 49.2)
- added R94: 10K, Resistor_SMD:R_0603_1608Metric, F.Cu at (269.9, 51.7)
- added R95: 10K, Resistor_SMD:R_0603_1608Metric, F.Cu at (269.9, 54.2)
- added R96: 10K, Resistor_SMD:R_0603_1608Metric, F.Cu at (269.9, 56.7)
- added R97: 470, Resistor_SMD:R_0603_1608Metric, F.Cu at (274.0, 44.2)
- added R98: 470, Resistor_SMD:R_0603_1608Metric, F.Cu at (274.0, 46.7)
- added R99: 470, Resistor_SMD:R_0603_1608Metric, F.Cu at (277.4, 56.6)
- added U10: 74LVC125, Package_DFN_QFN:DHVQFN-14-1EP_2.5x3mm_P0.5mm_EP1x1.5mm, F.Cu at (224.2, 74.2)
- added U11: THVD1420D, footprints:SOIC-8_4.9x3.91mm_P1.27mm, F.Cu at (225.4, 81.3)
- added U12: THVD1420D, footprints:SOIC-8_4.9x3.91mm_P1.27mm, F.Cu at (241.8, 83.2)
- added U13: 74LVC125, Package_DFN_QFN:DHVQFN-14-1EP_2.5x3mm_P0.5mm_EP1x1.5mm, F.Cu at (216.3, 98.5)
- added U14: 74HC595, Package_SO:TSSOP-16_4.4x5mm_P0.65mm, F.Cu at (193.8, 110.5)
- added U15: TPS274160BRLHR, Package_DFN_QFN:WQFN-28-1EP_4x4mm_P0.4mm_EP2.7x2.7mm_ThermalVias, F.Cu at (362.2, 25.1)
- added U16: 74HC595, Package_SO:TSSOP-16_4.4x5mm_P0.65mm, F.Cu at (377.7, 25.3)
- added U17: 74HC595, Package_SO:TSSOP-16_4.4x5mm_P0.65mm, F.Cu at (377.7, 31.9)
- added U18: 74HC595, Package_SO:TSSOP-16_4.4x5mm_P0.65mm, F.Cu at (324.4, 65.5)
- added U19: TPS274160BRLHR, Package_DFN_QFN:WQFN-28-1EP_4x4mm_P0.4mm_EP2.7x2.7mm_ThermalVias, F.Cu at (362.2, 31.4)
- added U20: 74HC595, Package_SO:TSSOP-16_4.4x5mm_P0.65mm, F.Cu at (324.4, 72.0)
- added U21: 74HC595, Package_SO:TSSOP-16_4.4x5mm_P0.65mm, F.Cu at (324.4, 78.6)
- added U22: TPS274160BRLHR, Package_DFN_QFN:WQFN-28-1EP_4x4mm_P0.4mm_EP2.7x2.7mm_ThermalVias, F.Cu at (362.2, 37.7)
- added U23: TPS274160BRLHR, Package_DFN_QFN:WQFN-28-1EP_4x4mm_P0.4mm_EP2.7x2.7mm_ThermalVias, F.Cu at (362.2, 44.0)
- added U24: 74HC595, Package_SO:TSSOP-16_4.4x5mm_P0.65mm, F.Cu at (299.8, 77.5)
- added U25: 74HC595, Package_SO:TSSOP-16_4.4x5mm_P0.65mm, F.Cu at (287.2, 82.7)
- added U26: 74HC595, Package_SO:TSSOP-16_4.4x5mm_P0.65mm, F.Cu at (290.9, 82.7)
- added U27: 74LVC125, Package_DFN_QFN:DHVQFN-14-1EP_2.5x3mm_P0.5mm_EP1x1.5mm, F.Cu at (287.7, 38.3)
- added U28: 74LVC125, Package_DFN_QFN:DHVQFN-14-1EP_2.5x3mm_P0.5mm_EP1x1.5mm, F.Cu at (292.5, 38.3)
- added U29: THVD1420D, footprints:SOIC-8_4.9x3.91mm_P1.27mm, F.Cu at (299.2, 31.1)
- added U30: THVD1420D, footprints:SOIC-8_4.9x3.91mm_P1.27mm, F.Cu at (302.9, 31.1)
- added U31: 74LVC125, Package_DFN_QFN:DHVQFN-14-1EP_2.5x3mm_P0.5mm_EP1x1.5mm, F.Cu at (266.3, 61.0)
- added U32: 74HC595, Package_SO:TSSOP-16_4.4x5mm_P0.65mm, F.Cu at (271.1, 61.0)
- added U33: 74HC595, Package_SO:TSSOP-16_4.4x5mm_P0.65mm, F.Cu at (277.8, 53.8)
- added U34: 74HC595, Package_SO:TSSOP-16_4.4x5mm_P0.65mm, F.Cu at (281.5, 53.8)
- added U35: 74LVC125, Package_DFN_QFN:DHVQFN-14-1EP_2.5x3mm_P0.5mm_EP1x1.5mm, F.Cu at (244.9, 61.0)
- added U36: 74LVC125, Package_DFN_QFN:DHVQFN-14-1EP_2.5x3mm_P0.5mm_EP1x1.5mm, F.Cu at (249.7, 61.0)
- added U37: THVD1420D, footprints:SOIC-8_4.9x3.91mm_P1.27mm, F.Cu at (256.4, 53.8)
- added U38: THVD1420D, footprints:SOIC-8_4.9x3.91mm_P1.27mm, F.Cu at (260.1, 53.8)
- added U39: 74LVC125, Package_DFN_QFN:DHVQFN-14-1EP_2.5x3mm_P0.5mm_EP1x1.5mm, F.Cu at (287.7, 61.0)
- added U40: 74HC595, Package_SO:TSSOP-16_4.4x5mm_P0.65mm, F.Cu at (292.5, 61.0)
- added U41: 74HC595, Package_SO:TSSOP-16_4.4x5mm_P0.65mm, F.Cu at (299.2, 53.8)
- added U42: 74HC595, Package_SO:TSSOP-16_4.4x5mm_P0.65mm, F.Cu at (302.9, 53.8)
- added U43: 74LVC125, Package_DFN_QFN:DHVQFN-14-1EP_2.5x3mm_P0.5mm_EP1x1.5mm, F.Cu at (266.3, 38.3)
- added U44: 74LVC125, Package_DFN_QFN:DHVQFN-14-1EP_2.5x3mm_P0.5mm_EP1x1.5mm, F.Cu at (271.1, 38.3)
- added U45: THVD1420D, footprints:SOIC-8_4.9x3.91mm_P1.27mm, F.Cu at (277.8, 31.1)
- added U46: THVD1420D, footprints:SOIC-8_4.9x3.91mm_P1.27mm, F.Cu at (281.5, 31.1)
- added U47: 74LVC125, Package_DFN_QFN:DHVQFN-14-1EP_2.5x3mm_P0.5mm_EP1x1.5mm, F.Cu at (244.9, 38.3)
- added U48: 74HC595, Package_SO:TSSOP-16_4.4x5mm_P0.65mm, F.Cu at (249.7, 38.3)
- added U49: 74HC595, Package_SO:TSSOP-16_4.4x5mm_P0.65mm, F.Cu at (256.4, 31.1)
- added U50: 74HC595, Package_SO:TSSOP-16_4.4x5mm_P0.65mm, F.Cu at (260.1, 31.1)
- added U51: 74HC595, Package_SO:TSSOP-16_4.4x5mm_P0.65mm, F.Cu at (328.5, 93.7)
- added U52: 74LVC125, Package_DFN_QFN:DHVQFN-14-1EP_2.5x3mm_P0.5mm_EP1x1.5mm, F.Cu at (328.5, 100.3)
- added U53: 74LVC125, Package_DFN_QFN:DHVQFN-14-1EP_2.5x3mm_P0.5mm_EP1x1.5mm, F.Cu at (328.5, 106.9)
- added U54: THVD1420D, footprints:SOIC-8_4.9x3.91mm_P1.27mm, F.Cu at (328.5, 113.5)
- added U55: THVD1420D, footprints:SOIC-8_4.9x3.91mm_P1.27mm, F.Cu at (328.5, 120.1)
- added U56: 74LVC125, Package_DFN_QFN:DHVQFN-14-1EP_2.5x3mm_P0.5mm_EP1x1.5mm, F.Cu at (337.6, 93.7)
- added U57: 74HC595, Package_SO:TSSOP-16_4.4x5mm_P0.65mm, F.Cu at (337.6, 100.3)
- added U58: 74HC595, Package_SO:TSSOP-16_4.4x5mm_P0.65mm, F.Cu at (337.6, 106.9)
- added U59: 74HC595, Package_SO:TSSOP-16_4.4x5mm_P0.65mm, F.Cu at (337.6, 113.5)
- added U60: 74LVC125, Package_DFN_QFN:DHVQFN-14-1EP_2.5x3mm_P0.5mm_EP1x1.5mm, F.Cu at (337.6, 120.1)
- added U61: 74LVC125, Package_DFN_QFN:DHVQFN-14-1EP_2.5x3mm_P0.5mm_EP1x1.5mm, F.Cu at (346.8, 93.7)
- added U62: THVD1420D, footprints:SOIC-8_4.9x3.91mm_P1.27mm, F.Cu at (346.8, 100.3)
- added U63: THVD1420D, footprints:SOIC-8_4.9x3.91mm_P1.27mm, F.Cu at (346.8, 106.9)
- added U64: 74LVC125, Package_DFN_QFN:DHVQFN-14-1EP_2.5x3mm_P0.5mm_EP1x1.5mm, F.Cu at (346.8, 113.5)
- added U65: TPS54202DDC, Package_TO_SOT_SMD:SOT-23-6, F.Cu at (289.1, 109.8)
- added U66: 74LVC125, Package_DFN_QFN:DHVQFN-14-1EP_2.5x3mm_P0.5mm_EP1x1.5mm, F.Cu at (218.2, 55.1)
- added U67: 74HC595, Package_SO:TSSOP-16_4.4x5mm_P0.65mm, F.Cu at (270.1, 100.6)
- added U68: 74HC595, Package_SO:TSSOP-16_4.4x5mm_P0.65mm, F.Cu at (270.1, 107.2)
- added U69: 74HC595, Package_SO:TSSOP-16_4.4x5mm_P0.65mm, F.Cu at (270.1, 113.8)
- added U70: 74LVC125, Package_DFN_QFN:DHVQFN-14-1EP_2.5x3mm_P0.5mm_EP1x1.5mm, F.Cu at (267.7, 120.1)
- added U71: 74LVC125, Package_DFN_QFN:DHVQFN-14-1EP_2.5x3mm_P0.5mm_EP1x1.5mm, F.Cu at (218.2, 47.5)
- added U72: THVD1420D, footprints:SOIC-8_4.9x3.91mm_P1.27mm, F.Cu at (251.1, 119.4)
- added U73: THVD1420D, footprints:SOIC-8_4.9x3.91mm_P1.27mm, F.Cu at (254.8, 119.4)
- added U74: 74LVC125, Package_DFN_QFN:DHVQFN-14-1EP_2.5x3mm_P0.5mm_EP1x1.5mm, F.Cu at (260.8, 142.8)
- added U75: 74HC595, Package_SO:TSSOP-16_4.4x5mm_P0.65mm, F.Cu at (254.0, 128.0)
- added U76: 74HC595, Package_SO:TSSOP-16_4.4x5mm_P0.65mm, F.Cu at (254.0, 134.6)
- added U77: 74HC595, Package_SO:TSSOP-16_4.4x5mm_P0.65mm, F.Cu at (254.0, 141.2)
- added U78: 74LVC125, Package_DFN_QFN:DHVQFN-14-1EP_2.5x3mm_P0.5mm_EP1x1.5mm, F.Cu at (265.5, 142.8)
- added U79: 74LVC125, Package_DFN_QFN:DHVQFN-14-1EP_2.5x3mm_P0.5mm_EP1x1.5mm, F.Cu at (225.0, 47.5)
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Connections:
- J1 pad 10: /FPGA Connector/IN_3 -> /FPGA Connector/OUT_3
- J1 pad 12: /FPGA Connector/IN_4 -> /FPGA Connector/OUT_4
- J1 pad 14: /FPGA Connector/IN_5 -> /FPGA Connector/OUT_5
- J1 pad 16: /FPGA Connector/IN_6 -> /FPGA Connector/OUT_6
- J1 pad 18: /FPGA Connector/IN_7 -> /FPGA Connector/OUT_7
- J1 pad 2: /FPGA Connector/IN_0 -> /FPGA Connector/OUT_0
- J1 pad 20: /FPGA Connector/IN_8 -> /FPGA Connector/OUT_8
- J1 pad 24: /FPGA Connector/IN_9 -> /FPGA Connector/OUT_9
- J1 pad 26: /FPGA Connector/IN_10 -> /FPGA Connector/OUT_10
- J1 pad 28: /FPGA Connector/IN_11 -> /FPGA Connector/OUT_11
- J1 pad 30: /FPGA Connector/IN_12 -> /FPGA Connector/OUT_12
- J1 pad 32: /FPGA Connector/IN_13 -> /FPGA Connector/OUT_13
- J1 pad 34: /FPGA Connector/IN_14 -> /FPGA Connector/OUT_14
- J1 pad 38: /FPGA Connector/IN_15 -> /FPGA Connector/OUT_15
- J1 pad 4: /FPGA Connector/IN_1 -> /FPGA Connector/OUT_1
- J1 pad 6: /FPGA Connector/IN_2 -> /FPGA Connector/OUT_2
- U1 pad 10: unconnected-(U1-PC2-Pad10) -> /MCU/5V_LOGIC_SENSE
- U1 pad 11: unconnected-(U1-PC3-Pad11) -> /MCU/5V_PORT_SENSE
- U1 pad 14: unconnected-(U1-PA0-Pad14) -> /MCU/HV_BANK_1_CURRENT_SENSE
- U1 pad 15: unconnected-(U1-PA1-Pad15) -> /MCU/HV_BANK_2_CURRENT_SENSE
- U1 pad 20: unconnected-(U1-PA4-Pad20) -> /MCU/PORT_1/2_VSENSE
- U1 pad 21: unconnected-(U1-PA5-Pad21) -> /MCU/PORT_3/4_VSENSE
- U1 pad 22: unconnected-(U1-PA6-Pad22) -> /MCU/PORT_5/6_VSENSE
- U1 pad 23: unconnected-(U1-PA7-Pad23) -> /MCU/PORT_7/8_VSENSE
- U1 pad 24: unconnected-(U1-PC4-Pad24) -> /MCU/LV_BANK_1_CURRENT_SENSE
- U1 pad 25: unconnected-(U1-PC5-Pad25) -> /MCU/LV_BANK_2_CURRENT_SENSE
- U1 pad 26: /MCU/VCXO_TRIM -> unconnected-(U1-PB0-Pad26)
- U1 pad 39: unconnected-(U1-PC8-Pad39) -> /MCU/VCXO_TRIM
- U1 pad 4: unconnected-(U1-PC15-Pad4) -> /MCU/CONFIG_UPDATE
- U1 pad 40: unconnected-(U1-PC9-Pad40) -> /MCU/CONFIG_CLR_N
- U1 pad 51: unconnected-(U1-PC10-Pad51) -> /MCU/CONFIG_CLK
- U1 pad 52: unconnected-(U1-PC11-Pad52) -> /MCU/CONFIG_OE_N
- U1 pad 53: unconnected-(U1-PC12-Pad53) -> /MCU/CONFIG_DATA
- U2 pad 1: /FPGA Connector/IO_1 -> /FPGA Connector/IN_1
- U2 pad 3: /FPGA Connector/IO_2 -> /FPGA Connector/IN_2
- U2 pad 4: /FPGA Connector/IO_3 -> /FPGA Connector/IN_3
- U2 pad 6: /FPGA Connector/IO_0 -> /FPGA Connector/IN_0
- U3 pad 1: /FPGA Connector/IO_5 -> /FPGA Connector/IN_5
- U3 pad 3: /FPGA Connector/IO_6 -> /FPGA Connector/IN_6
- U3 pad 4: /FPGA Connector/IO_7 -> /FPGA Connector/IN_7
- U3 pad 6: /FPGA Connector/IO_4 -> /FPGA Connector/IN_4
- U4 pad 1: /FPGA Connector/IO_9 -> /FPGA Connector/IN_9
- U4 pad 3: /FPGA Connector/IO_10 -> /FPGA Connector/IN_10
- U4 pad 4: /FPGA Connector/IO_11 -> /FPGA Connector/IN_11
- U4 pad 6: /FPGA Connector/IO_8 -> /FPGA Connector/IN_8
- U5 pad 1: /FPGA Connector/IO_13 -> /FPGA Connector/IN_13
- U5 pad 3: /FPGA Connector/IO_14 -> /FPGA Connector/IN_14
- U5 pad 4: /FPGA Connector/IO_15 -> /FPGA Connector/IN_15
- U5 pad 6: /FPGA Connector/IO_12 -> /FPGA Connector/IN_12
