File: KiCad/Serial Module/port_power.kicad_sch (KiCad schematic)
At the start: 50 parts, among them Q1 Q_NMOS_GDS, Q10 Q_NMOS_GDS, Q2 Q_NMOS_GDS, Q5 Q_NMOS_GDS, Q6 Q_NMOS_GDS, Q7 Q_NMOS_GDS, Q8 Q_NMOS_GDS, Q9 Q_NMOS_GDS, U18 INA180A1, U20 FAN7842, U21 FAN7842, U22 FAN7842, U23 FAN7842

Commit message: update serial module and backplane hw
Parts:
- removed C25, C26: 0.1uf, symbol Device:C
- removed C29, C31, C32, C34: C, symbol Device:C
- removed D10: SMAJ24A, Diode_SMD:D_SMA, symbol Diode:SMAJ24A
- removed D11: D_Zener, symbol Device:D_Zener
- removed F1: 1A, symbol Device:Polyfuse
- removed Q1, Q10, Q2, Q5, Q6, Q7, Q8, Q9: Q_NMOS_GDS, symbol Device:Q_NMOS_GDS
- removed R38, R39, R45, R46, R47: R, symbol Device:R
- removed R44, R48, R49, R50: 10, symbol Device:R
- removed U18: INA180A1, Package_TO_SOT_SMD:SOT-23-5, symbol Amplifier_Current:INA180A1
- removed U20, U21, U22, U23: FAN7842, Package_SO:SOIC-8_3.9x4.9mm_P1.27mm, symbol Driver_FET:FAN7842
- added C110, C115, C116, C132, C136, C137, C36, C46, C47, C48, C49: 22uf, Capacitor_SMD:C_1206_3216Metric, symbol Device:C
- added C112, C113, C133, C134: .1uf, Capacitor_SMD:C_0402_1005Metric, symbol Device:C
- added C114, C135: 75pf, Capacitor_SMD:C_0402_1005Metric, symbol Device:C
- added C138, C139, C149, C38, C42, C43, C52, C53: .1uf, Capacitor_SMD:C_0603_1608Metric, symbol Device:C
- added C20, C21, C22, C37, C39, C40, C41, C50, C51, C54, C55, C56, C57, C58, C59: 22nf, Capacitor_SMD:C_0603_1608Metric, symbol Device:C
- added C29, C34, C44, C45: 120uf, Capacitor_SMD:CP_Elec_8x10.5, symbol Device:C_Polarized
- added D10, D11, D24, D25, D26, D27, D8, D9: D_Schottky, Diode_SMD:D_SOD-123F, symbol Device:D_Schottky
- added D50, D51: BAT54SLT1G, Package_TO_SOT_SMD:SOT-23, symbol Device:D_Dual_Series_AKC
- added JP1, JP2, JP3, JP4: Jumper_3_Bridged12, Connector_PinHeader_2.54mm:PinHeader_1x03_P2.54mm_Vertical, symbol Jumper:Jumper_3_Bridged12
- added L1, L5: 15uH, footprints:FCH0650, symbol Device:L
- added R160, R161, R24, R243, R244, R247, R248, R26, R27, R28: 10k, Resistor_SMD:R_0603_1608Metric, symbol Device:R
- added R162, R245: 100k, Resistor_SMD:R_0402_1005Metric, symbol Device:R_US
- added R163: 12.4k, Resistor_SMD:R_0402_1005Metric, symbol Device:R_US
- added R246: 13.3k, Resistor_SMD:R_0402_1005Metric, symbol Device:R_US
- added U14, U18, U20, U21, U84: 74HC595, Package_SO:TSSOP-16_4.4x5mm_P0.65mm, symbol 74xx:74HC595
- added U15, U19, U22, U23: TPS274160BRLHR, Package_DFN_QFN:WQFN-28-1EP_4x4mm_P0.4mm_EP2.7x2.7mm_ThermalVias, symbol TPS274160B:TPS274160BRLHR
- added U65, U82: TPS54202DDC, Package_TO_SOT_SMD:SOT-23-6, symbol Regulator_Switching:TPS54202DDC
- C23: value C -> 22nf; footprint (none) -> Capacitor_SMD:C_0603_1608Metric
- C24, C28, C35: value C -> 22uf; footprint (none) -> Capacitor_SMD:C_1206_3216Metric; Generic Allowed? (none) -> yes; LCSC# (none) -> C12891; Manufacturer (none) -> Samsung Electro-Mechanics; Part number (none) -> CL31A226KAHNNNE; cost (none) -> 0.04
- C27, C30, C33: value 0.1uf -> .1uf; footprint (none) -> Capacitor_SMD:C_0603_1608Metric
- D12, D13, D14, D15, D16, D17, D18, D19, D20, D21, D22, D23: footprint (none) -> Diode_SMD:D_SOD-123F; LCSC# (none) -> C908664; Manufacturer (none) -> GOODWORK; Part Number (none) -> K24
Connections:
- net +24V_PORT: now also JP1.1 (A), JP2.1 (A); no longer D19.1 (K), D22.2 (A)
- net +3.3V: now also C30.1, C33.1, C149.1, C42.1, C43.1, D50.2 (K), D51.2 (K), R24.1, R26.1, R27.1, R28.1, U14.16 (VCC), U18.16 (VCC), U20.16 (VCC), U21.16 (VCC), U84.16 (VCC)
- net +5V_PORT: now also C114.2, C115.2, C116.2, JP3.1 (A), JP4.1 (A), L5.2, R160.1, R162.2; no longer D16.2 (A), D17.1 (K)
- net GND: now also C23.2, C24.1, C28.1, C35.1, D12.2 (A), D14.2 (A), D20.2 (A), D21.2 (A), C110.1, C112.1, C115.1, C116.1, C132.1, C133.1, C136.1, C137.1, C138.2, C139.2, C149.2, C20.2, C21.2, C22.2, C29.2, C34.2, C36.1, C37.2, C38.2, C39.2, C40.2, C41.2, C42.2, C43.2, C44.2, C45.2, C46.1, C47.1, C48.1, C49.1, C50.2, C51.2, C52.2, C53.2, C54.2, C55.2, C56.2, C57.2, C58.2, C59.2, D50.1 (A), D51.1 (A), R161.2, R163.1, R244.2, R246.1, R247.1, R248.1, U14.8 (GND), U15.26 (GND), U15.29 (PowerPAD), U15.9 (GND), U18.8 (GND), U19.26 (GND), U19.29 (PowerPAD), U19.9 (GND), U20.8 (GND), U21.8 (GND), U22.26 (GND), U22.29 (PowerPAD), U22.9 (GND), U23.26 (GND), U23.29 (PowerPAD), U23.9 (GND), U65.1 (GND), U82.1 (GND), U84.8 (GND)
- net PORT_8+: now reaches D13.1 (K)
- net PORT_8+: now also D19.1 (K); no longer C24.1
- net at C24.2: now also C27.1, C28.2, D12.1 (K), C29.1, JP1.2 (C), U15.17 (VS), U15.18 (VS), U15.19 (VS), U15.20 (VS); no longer D14.2 (A)
- net at D20.1 (K): now also C44.1, C46.2, C48.2, C52.1, JP3.2 (C), U22.17 (VS), U22.18 (VS), U22.19 (VS), U22.20 (VS); no longer D21.2 (A)
- net PORT_7+: now reaches D23.1 (K)
- net PORT_7+: now also D15.1 (K); no longer C35.1
- net at C35.2: now also D14.1 (K), C34.1, C36.2, C38.1, JP2.2 (C), U19.17 (VS), U19.18 (VS), U19.19 (VS), U19.20 (VS); no longer D19.2 (A)
- net at D17.2 (A): now also C41.1, U19.24 (OUT1), U19.25 (OUT1); no longer C28.2
- net at D23.2 (A): now also C55.1, U23.14 (OUT3), U23.15 (OUT3); no longer D22.1 (K)
- net at D18.2 (A): now also C50.1, U22.12 (OUT4), U22.13 (OUT4)
- net at D21.1 (K): now also C45.1, C47.2, C49.2, C53.1, JP4.2 (C), U23.17 (VS), U23.18 (VS), U23.19 (VS), U23.20 (VS)
- net at D15.2 (A): now also C39.1, U19.14 (OUT3), U19.15 (OUT3); no longer D16.1 (K)
- removed net +12V_PORT: C27.1, C30.1, C33.1, D18.1 (K), D20.2 (A)
- new net: C56.1, D24.2 (A), U22.22 (OUT2), U22.23 (OUT2)
- new net: C23.1, D11.2 (A), U15.24 (OUT1), U15.25 (OUT1)
- new net: C51.1, D19.2 (A), U23.12 (OUT4), U23.13 (OUT4)
- new net: U20.1 (QB), U22.28 (EN2)
- new net: U18.9 (QH'), U20.14 (SER)
- new net: U20.15 (QA), U22.27 (EN1)
- new net: U20.2 (QC), U22.1 (EN3)
- new net: U20.3 (QD), U22.2 (EN4)
- new net: U20.4 (QE), U22.3 (SEH)
- new net: U20.5 (QF), U22.4 (SEL)
- new net: U20.6 (QG), U22.11 (DIAG_EN)
- new net: U20.7 (QH), U22.10 (THER)
- new net: U20.9 (QH'), U21.14 (SER)
- new net: C37.1, D13.2 (A), U19.12 (OUT4), U19.13 (OUT4)
- new net: R24.2, U15.5 (FAULT_N)
- new net: U21.1 (QB), U23.28 (EN2)
- new net: U21.15 (QA), U23.27 (EN1)
- new net: U21.2 (QC), U23.1 (EN3)
- new net: U21.3 (QD), U23.2 (EN4)
- new net: U21.4 (QE), U23.3 (SEH)
- new net: U21.5 (QF), U23.4 (SEL)
- new net: U21.6 (QG), U23.11 (DIAG_EN)
- new net: U21.7 (QH), U23.10 (THER)
- new net: U21.9 (QH'), U84.14 (SER)
- new net: U14.2 (QC), U15.1 (EN3)
- new net: U14.7 (QH), U15.10 (THER)
- new net: U14.6 (QG), U15.11 (DIAG_EN)
- new net: C20.1, D8.2 (A), U15.12 (OUT4), U15.13 (OUT4)
- new net: C21.1, D9.2 (A), U15.14 (OUT3), U15.15 (OUT3)
- new net: U14.3 (QD), U15.2 (EN4)
- new net: C22.1, D10.2 (A), U15.22 (OUT2), U15.23 (OUT2)
- new net: U14.15 (QA), U15.27 (EN1)
- new net: U14.1 (QB), U15.28 (EN2)
- new net: U14.4 (QE), U15.3 (SEH)
- new net: U14.5 (QF), U15.4 (SEL)
- new net: C54.1, D22.2 (A), U22.14 (OUT3), U22.15 (OUT3)
- new net: C134.1, U82.6 (BOOT)
- new net: C134.2, L1.1, U82.2 (SW)
- new net: C58.1, D26.2 (A), U22.24 (OUT1), U22.25 (OUT1)
- new net: C135.1, R245.1, R246.2, U82.4 (FB)
- new net: C114.1, R162.1, R163.2, U65.4 (FB)
- new net: C59.1, D27.2 (A), U23.24 (OUT1), U23.25 (OUT1)
- new net: C40.1, D16.2 (A), U19.22 (OUT2), U19.23 (OUT2)
- new net: C57.1, D25.2 (A), U23.22 (OUT2), U23.23 (OUT2)
- new net: R28.2, U23.5 (FAULT_N)
- new net: C113.2, L5.1, U65.2 (SW)
- new net: C113.1, U65.6 (BOOT)
- new net: R27.2, U22.5 (FAULT_N)
- new net: U14.9 (QH'), U18.14 (SER)
- new net: U18.1 (QB), U19.28 (EN2)
- new net: U18.15 (QA), U19.27 (EN1)
- new net: U18.2 (QC), U19.1 (EN3)
- new net: U18.3 (QD), U19.2 (EN4)
- new net: U18.4 (QE), U19.3 (SEH)
- new net: U18.5 (QF), U19.4 (SEL)
- new net: U18.6 (QG), U19.11 (DIAG_EN)
- new net: U18.7 (QH), U19.10 (THER)
- new net: R26.2, U19.5 (FAULT_N)
- new net +24V: C110.2, C112.2, C132.2, C133.2, U65.3 (VIN), U82.3 (VIN)
- new net +5V_LOGIC: C135.2, C136.2, C137.2, L1.2, R243.1, R245.2
- new net +AUX_VH_PORT_BANK_1: JP1.3 (B)
- new net +AUX_VH_PORT_BANK_2: JP2.3 (B)
- new net +AUX_VL_PORT_BANK_1: JP3.3 (B)
- new net +AUX_VL_PORT_BANK_2: JP4.3 (B)
- new net 5V_LOGIC_VSENSE: C139.1, D51.3 (common), R243.2, R244.1
- new net 5V_PORT_VSENSE: C138.1, D50.3 (common), R160.2, R161.1
- new net CONFIG_CLK: U14.11 (SRCLK), U18.11 (SRCLK), U20.11 (SRCLK), U21.11 (SRCLK), U84.11 (SRCLK)
- new net CONFIG_CLR_N: U14.10 (~{SRCLR}), U18.10 (~{SRCLR}), U20.10 (~{SRCLR}), U21.10 (~{SRCLR}), U84.10 (~{SRCLR})
- new net CONFIG_DATA_IN: U14.14 (SER)
- new net CONFIG_OE_N: U14.13 (~{OE}), U18.13 (~{OE}), U20.13 (~{OE}), U21.13 (~{OE}), U84.13 (~{OE})
- new net CONFIG_UPDATE: U14.12 (RCLK), U18.12 (RCLK), U20.12 (RCLK), U21.12 (RCLK), U84.12 (RCLK)
- new net CURRENT_LIM_HV_BANK_1: U15.7 (CL)
- new net CURRENT_LIM_HV_BANK_2: U19.7 (CL)
- new net CURRENT_LIM_LV_BANK_1: U22.7 (CL)
- new net CURRENT_LIM_LV_BANK_2: U23.7 (CL)
- new net CURRENT_SENSE_HV_BANK_1: U15.6 (CS)
- new net CURRENT_SENSE_HV_BANK_2: U19.6 (CS)
- new net CURRENT_SENSE_LV_BANK_1: U22.6 (CS)
- new net CURRENT_SENSE_LV_BANK_2: U23.6 (CS)
- new net LOGIC_5V_POWER_EN: R248.2, U82.5 (EN), U84.1 (QB)
- new net PORT_1+: D11.1 (K), D26.1 (K)
- new net PORT_2+: D10.1 (K), D24.1 (K)
- new net PORT_3+: D22.1 (K), D9.1 (K)
- new net PORT_4+: D18.1 (K), D8.1 (K)
- new net PORT_5+: D17.1 (K), D27.1 (K)
- new net PORT_5V_POWER_EN: R247.2, U65.5 (EN), U84.15 (QA)
- new net PORT_6+: D16.1 (K), D25.1 (K)
- new net Port Vsense Mux/SELECT: U84.2 (QC)
Other:
- added sheet Port Vsense Mux (port_vsense_mux.kicad_sch)
- added sheet Port Vsense Mux1 (port_vsense_mux.kicad_sch)
- added sheet Port Vsense Mux2 (port_vsense_mux.kicad_sch)
- added sheet Port Vsense Mux3 (port_vsense_mux.kicad_sch)
- note added: "5V_PORT is set to ~5.4v to account for diode and wire drop"

Commit message: add current limit and sense parts, add possible endat solution
Parts:
- added C153, C154, C155, C156: 10nf, Capacitor_SMD:C_0603_1608Metric, symbol Device:C
- added D52, D53, D54, D55: BAT54SLT1G, Package_TO_SOT_SMD:SOT-23, symbol Device:D_Dual_Series_AKC
- added R249, R250, R251, R252: 330, Resistor_SMD:R_0603_1608Metric, symbol Device:R
Connections:
- net +3.3V: now also D52.2 (K), D53.2 (K), D54.2 (K), D55.2 (K)
- net CURRENT_SENSE_HV_BANK_1: now also C156.1, D52.3 (common), R249.1
- net CURRENT_SENSE_HV_BANK_2: now also C153.1, D53.3 (common), R250.1
- net CURRENT_SENSE_LV_BANK_1: now also C154.1, D55.3 (common), R252.1
- net CURRENT_SENSE_LV_BANK_2: now also C155.1, D54.3 (common), R251.1
- net GND: now also C153.2, C154.2, C155.2, C156.2, D52.1 (A), D53.1 (A), D54.1 (A), D55.1 (A), R249.2, R250.2, R251.2, R252.2
- net Current Limit Mux1/DATA_IN: now reaches U20.9 (QH')
- net Current Limit Mux1/DATA_IN: no longer U21.14 (SER)
- net FAULT_N_VH_BANK_1: now reaches R24.2, U15.5 (FAULT_N)
- net FAULT_N_VL_BANK_2: now reaches R28.2, U23.5 (FAULT_N)
- net FAULT_N_VL_BANK_1: now reaches R27.2, U22.5 (FAULT_N)
- net Current Limit Mux/DATA_IN: now reaches U14.9 (QH')
- net Current Limit Mux/DATA_IN: no longer U18.14 (SER)
- net FAULT_N_VH_BANK_2: now reaches R26.2, U19.5 (FAULT_N)
- net CURRENT_LIM_HV_BANK_1 renamed Current Limit Mux/CL_1
- net CURRENT_LIM_HV_BANK_2 renamed Current Limit Mux/CL_2
- net CURRENT_LIM_LV_BANK_1 renamed Current Limit Mux1/CL_1
- net CURRENT_LIM_LV_BANK_2 renamed Current Limit Mux1/CL_2
- new net Current Limit Mux/DATA_OUT: U18.14 (SER)
- new net Current Limit Mux1/DATA_OUT: U21.14 (SER)
Other:
- added sheet Current Limit Mux (current_limit_mux.kicad_sch)
- added sheet Current Limit Mux1 (current_limit_mux.kicad_sch)
- note added: "place cap near MCU"
- moved on the sheet: C149, C20, C21, C22, C23, C24, C27, C28, C29, C30, C33, C34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
