File: KiCad/Serial Module/port_power.kicad_sch (KiCad schematic)
At the start: 116 parts, among them U14 74HC595, U15 TPS274160BRLHR, U18 74HC595, U19 TPS274160BRLHR, U20 74HC595, U21 74HC595, U22 TPS274160BRLHR, U23 TPS274160BRLHR, U65 TPS54202DDC, U82 TPS54202DDC, U84 74HC595

Commit message: Serial Module: review fixes, full BOM part numbers, stock footprints
Schematic fixes:
- +24V_PORT tied to +24V; STM32 VBAT tied to VDD
- Pull-ups on CONFIG15-18 and on bias-buffer OE inputs; pull-downs on PC13/PC14
- CONFIG_UPDATE moved from PC15 to PC7; VCXO Vcon biased to 1.65 V
- RJ45 LED anodes moved from 5V_LOGIC to 3.3V
- 74LVC125 units kept within one transceiver-pair instance; fixed pair-1
  annotation (U27/U28 units) that shorted MUX_B to DI_B in the netlist
- 5 V bias buffers changed to TI SN74ACT125PWR (TTL inputs, 4.5-5.5 V)
- Current-limit NMOS changed to AO3400A (Transistor_FET symbol, SOT-23 G/S/D)
- 24 V input TVS changed to TI TVS2700DRVR flat-clamp (27 V standoff,
  35 V max clamp at 40 A) replacing PTVS26VZ1USK (42 V clamp)
- Removed unused port_vsense_muc.kicad_sch

BOM and footprints:
- Every part now has Manufacturer, Part number and LCSC# (verified in stock);
  YAGEO caps/resistors, TI logic where stocked
- 24 V-rail MLCCs now 10 uF 50 V X7R 1210; bulk caps 100 uF 50 V
- TPS274160B footprint corrected to VQFN-28 4x5 mm (RLH); THVD1420 to
  150-mil SOIC-8; all custom footprints replaced with KiCad stock except
  J1 (card connector) and J3 (2x4 RJ45)
- "Part Number" fields normalised to "Part number"

Co-Authored-By: Claude Opus 5.5 <noreply@anthropic.com>
Parts:
- added D56, D57: TVS2700, Package_SON:WSON-6-1EP_2x2mm_P0.65mm_EP1x1.6mm, symbol Power_Protection:TVS2700DRV
- added R389, R390, R391, R392, R393, R394, R395, R396, R397, R398, R399, R400, R401, R402, R403, R404: 10k, Resistor_SMD:R_0603_1608Metric, symbol Device:R
- C110, C132: value 22uf -> 10uF; footprint Capacitor_SMD:C_1206_3216Metric -> Capacitor_SMD:C_1210_3225Metric; Generic Allowed? yes -> (none); LCSC# C12891 -> C596319; Manufacturer Samsung Electro-Mechanics -> YAGEO; Part number CL31A226KAHNNNE -> CC1210KKX7R9BB106; cost 0.04 -> (none)
- C138, C139, C149, C27, C30, C33, C38, C42, C43, C52, C53: LCSC# (none) -> C14663; Manufacturer (none) -> YAGEO; Part number (none) -> CC0603KRX7R9BB104
- C153, C154, C155, C156: LCSC# (none) -> C100042; Manufacturer (none) -> YAGEO; Part number (none) -> CC0603KRX7R9BB103
- C20, C21, C22, C23, C37, C39, C40, C41, C50, C51, C54, C55, C56, C57, C58, C59: LCSC# (none) -> C106222; Manufacturer (none) -> YAGEO; Part number (none) -> CC0603KRX7R9BB223
- C24, C28, C35, C36: value 22uf -> 10uF; footprint Capacitor_SMD:C_1206_3216Metric -> Capacitor_SMD:C_1210_3225Metric; LCSC# C12891 -> C596319; Manufacturer Samsung Electro-Mechanics -> YAGEO; Part number CL31A226KAHNNNE -> CC1210KKX7R9BB106; cost 0.04 -> 0.3958
- C29, C34, C44, C45: value 120uf -> 100uF; LCSC# (none) -> C48935404; Manufacturer (none) -> jieerrui; Part number (none) -> RVE50V100M8X10
- D10, D11, D12, D13, D14, D15, D16, D17, D18, D19, D20, D21, D22, D23, D24, D25, D26, D27, D8, D9: Part Number K24 -> (none); Part number (none) -> K24
- JP1, JP2, JP3, JP4: LCSC# (none) -> C2937625; Manufacturer (none) -> XFCN; Part number (none) -> PZ254V-11-03P
- L1, L5: footprint footprints:FCH0650 -> Inductor_SMD:L_Changjiang_FXL0650; LCSC# C20415538 -> C475522; Manufacturer FANGCHENG -> cjiang (Changjiang Microelectronics); Part number CY54-15UH -> FXL0650-150-M; cost 0.05 -> 0.1258
- R160, R161, R24, R243, R244, R247, R248, R26, R27, R28: LCSC# (none) -> C98220; Manufacturer (none) -> YAGEO; Part number (none) -> RC0603FR-0710KL
- R163: Generic Allowed? yes, 1% or better -> (none); LCSC# C274352 -> C138060; Part number RC0402FR-0713K3L -> RC0402FR-0712K4L; cost 0.0007 -> (none)
- R249, R250, R251, R252: LCSC# (none) -> C105881; Manufacturer (none) -> YAGEO; Part number (none) -> RC0603FR-07330RL
- U14, U18, U20, U21, U84: LCSC# C5948 -> C273642; Manufacturer (none) -> TI; Part number (none) -> SN74HC595PWR
- U15, U19, U22, U23: footprint Package_DFN_QFN:WQFN-28-1EP_4x4mm_P0.4mm_EP2.7x2.7mm_ThermalVias -> Package_DFN_QFN:VQFN-28-1EP_4x5mm_P0.5mm_EP2.55x3.55mm_ThermalVias; Part number (none) -> TPS274160BRLHR
Connections:
- net +24V_PORT is gone; now on net +24V: JP1.1 (A), JP2.1 (A)
- net +24V: now also C110.1, C132.1, D56.4 (IN), D56.5 (IN), D56.6 (IN), D57.4 (IN), D57.5 (IN), D57.6 (IN); no longer C110.2, C132.2
- net GND: now also C110.2, C132.2, D56.1 (GND), D56.2 (GND), D56.3 (GND), D56.7 (GND), D57.1 (GND), D57.2 (GND), D57.3 (GND), D57.7 (GND); no longer C110.1, C132.1
- net at U20.1 (QB): now also R390.1; no longer U22.28 (EN2)
- net at U20.15 (QA): now also R389.1; no longer U22.27 (EN1)
- net at U20.2 (QC): now also R391.1; no longer U22.1 (EN3)
- net at U20.3 (QD): now also R392.1; no longer U22.2 (EN4)
- net at U21.1 (QB): now also R394.1; no longer U23.28 (EN2)
- net at U21.15 (QA): now also R393.1; no longer U23.27 (EN1)
- net at U21.2 (QC): now also R395.1; no longer U23.1 (EN3)
- net at U21.3 (QD): now also R396.1; no longer U23.2 (EN4)
- net at U15.1 (EN3): now also R403.2; no longer U14.2 (QC)
- net at U15.2 (EN4): now also R404.2; no longer U14.3 (QD)
- net at U14.15 (QA): now also R401.1; no longer U15.27 (EN1)
- net at U14.1 (QB): now also R402.1; no longer U15.28 (EN2)
- net at U18.1 (QB): now also R398.1; no longer U19.28 (EN2)
- net at U18.15 (QA): now also R397.1; no longer U19.27 (EN1)
- net at U18.2 (QC): now also R399.1; no longer U19.1 (EN3)
- net at U18.3 (QD): now also R400.1; no longer U19.2 (EN4)
- new net: R402.2, U15.28 (EN2)
- new net: R395.2, U23.1 (EN3)
- new net: R401.2, U15.27 (EN1)
- new net: R400.2, U19.2 (EN4)
- new net: R393.2, U23.27 (EN1)
- new net: R392.2, U22.2 (EN4)
- new net: R394.2, U23.28 (EN2)
- new net: R403.1, U14.2 (QC)
- new net: R404.1, U14.3 (QD)
- new net: R397.2, U19.27 (EN1)
- new net: R396.2, U23.2 (EN4)
- new net: R390.2, U22.28 (EN2)
- new net: R399.2, U19.1 (EN3)
- new net: R398.2, U19.28 (EN2)
- new net: R389.2, U22.27 (EN1)
- new net: R391.2, U22.1 (EN3)
Other:
- moved on the sheet: C112, C133
