File: KiCad/Serial Module/transceivers.kicad_sch (KiCad schematic)
At the start: 9 parts, among them Q3 Q_NMOS_GDS, Q4 Q_NMOS_GDS, U13 TCA9555PWR, U19 FAN7842

Commit message: update serial module and backplane hw
Parts:
- removed C22: C, symbol Device:C
- removed Q3, Q4: Q_NMOS_GDS, symbol Device:Q_NMOS_GDS
- removed R40, R41: 100, symbol Device:R
- removed R42, R43: 10k, symbol Device:R
- removed U13: TCA9555PWR, Package_SO:TSSOP-24_4.4x7.8mm_P0.65mm, symbol Interface_Expansion:TCA9555PWR
- removed U19: FAN7842, Package_SO:SOIC-8_3.9x4.9mm_P1.27mm, symbol Driver_FET:FAN7842
- added J3: ~, footprints:RJ45-TH_HC-RJ45-059D-2X4-2-04, symbol HC-RJ45-059D-2x4-2-04:HC-RJ45-059D-2*4-2-04
- added R45, R46, R47, R48, R49, R50, R51, R52, R53, R54, R55, R56, R57, R58, R59, R60: 1k, Resistor_SMD:R_0603_1608Metric, symbol Device:R
Connections:
- net GND: now also J3.10, J3.16, J3.2, J3.26, J3.32, J3.34, J3.40, J3.50, J3.56, J3.58, J3.64, J3.74, J3.8, J3.80, J3.82, J3.88, J3.SH, J3.SH, J3.SH, J3.SH, J3.SH, J3.SH, J3.SH, J3.SH
- new net: J3.66, R56.1
- new net: J3.46, R50.1
- new net: J3.48, R49.1
- new net: J3.90, R60.1
- new net: J3.92, R59.1
- new net: J3.22, R46.1
- new net: J3.72, R53.1
- new net: J3.24, R45.1
- new net: J3.96, R57.1
- new net: J3.68, R55.1
- new net: J3.70, R54.1
- new net: J3.94, R58.1
- new net: J3.44, R51.1
- new net: J3.18, R48.1
- new net: J3.42, R52.1
- new net: J3.20, R47.1
- new net +5V_LOGIC: R45.2, R46.2, R47.2, R48.2, R49.2, R50.2, R51.2, R52.2, R53.2, R54.2, R55.2, R56.2, R57.2, R58.2, R59.2, R60.2
- new net PORT_1+: J3.1, J3.7
- new net PORT_1_DATA_1+: J3.3
- new net PORT_1_DATA_1-: J3.6
- new net PORT_1_DATA_2+: J3.5
- new net PORT_1_DATA_2-: J3.4
- new net PORT_1_LED_GRN: J3.21
- new net PORT_1_LED_YLW: J3.23
- new net PORT_2+: J3.15, J3.9
- new net PORT_2_DATA_1+: J3.11
- new net PORT_2_DATA_1-: J3.14
- new net PORT_2_DATA_2+: J3.13
- new net PORT_2_DATA_2-: J3.12
- new net PORT_2_LED_GRN: J3.17
- new net PORT_2_LED_YLW: J3.19
- new net PORT_3+: J3.25, J3.31
- new net PORT_3_DATA_1+: J3.27
- new net PORT_3_DATA_1-: J3.30
- new net PORT_3_DATA_2+: J3.29
- new net PORT_3_DATA_2-: J3.28
- new net PORT_3_LED_GRN: J3.45
- new net PORT_3_LED_YLW: J3.47
- new net PORT_4+: J3.33, J3.39
- new net PORT_4_DATA_1+: J3.35
- new net PORT_4_DATA_1-: J3.38
- new net PORT_4_DATA_2+: J3.37
- new net PORT_4_DATA_2-: J3.36
- new net PORT_4_LED_GRN: J3.41
- new net PORT_4_LED_YLW: J3.43
- new net PORT_5+: J3.49, J3.55
- new net PORT_5_DATA_1+: J3.51
- new net PORT_5_DATA_1-: J3.54
- new net PORT_5_DATA_2+: J3.53
- new net PORT_5_DATA_2-: J3.52
- new net PORT_5_LED_GRN: J3.69
- new net PORT_5_LED_YLW: J3.71
- new net PORT_6+: J3.57, J3.63
- new net PORT_6_DATA_1+: J3.59
- new net PORT_6_DATA_1-: J3.62
- new net PORT_6_DATA_2+: J3.61
- new net PORT_6_DATA_2-: J3.60
- new net PORT_6_LED_GRN: J3.65
- new net PORT_6_LED_YLW: J3.67
- new net PORT_7+: J3.73, J3.79
- new net PORT_7_DATA_1+: J3.75
- new net PORT_7_DATA_1-: J3.78
- new net PORT_7_DATA_2+: J3.77
- new net PORT_7_DATA_2-: J3.76
- new net PORT_7_LED_GRN: J3.93
- new net PORT_7_LED_YLW: J3.95
- new net PORT_8+: J3.81, J3.87
- new net PORT_8_DATA_1+: J3.83
- new net PORT_8_DATA_1-: J3.86
- new net PORT_8_DATA_2+: J3.85
- new net PORT_8_DATA_2-: J3.84
- new net PORT_8_LED_GRN: J3.89
- new net PORT_8_LED_YLW: J3.91
Other:
- added sheet Transceiver pair2 (transceiver_pair.kicad_sch)
- added sheet Transceiver pair3 (transceiver_pair.kicad_sch)
- added sheet Transceiver pair4 (transceiver_pair.kicad_sch)
- added sheet Transceiver pair5 (transceiver_pair.kicad_sch)
- added sheet Transceiver pair6 (transceiver_pair.kicad_sch)
- added sheet Transceiver pair7 (transceiver_pair.kicad_sch)
- sheet Port Power ports: added 5V_LOGIC_VSENSE, 5V_PORT_VSENSE, CONFIG_CLK, CONFIG_CLR_N, CONFIG_DATA_IN, CONFIG_OE_N, CONFIG_UPDATE, CURRENT_SENSE_HV_BANK_1, CURRENT_SENSE_HV_BANK_2, CURRENT_SENSE_LV_BANK_1, CURRENT_SENSE_LV_BANK_2, PORT_1+, PORT_1/2_VSENSE, PORT_2+, PORT_3+, PORT_3/4_VSENSE, PORT_4+, PORT_5+, PORT_5/6_VSENSE, PORT_6+, PORT_7+, PORT_7/8_VSENSE, PORT_8+; removed 12V_ENABLE, 12V_SQUARE, 24V_ENABLE, 5V_ENABLE, CURRENT_SENSE, MAIN_ENABLE, PORT+A, PORT-A
- sheet Transceiver pair ports: added CONFIG_CLK, CONFIG_CLR_N, CONFIG_DATA_IN, CONFIG_DATA_OUT, CONFIG_OE_N, CONFIG_UPDATE, FPGA_MUX_IN_A, FPGA_MUX_IN_B, FPGA_MUX_OUT_A, FPGA_MUX_OUT_B, LED_GRN, LED_YLW; removed 1BIAS+, 1BIAS-, 2BIAS+, 2BIAS-, CONFIG1, CONFIG10, CONFIG2, CONFIG3, CONFIG4, CONFIG5, CONFIG6, CONFIG7, CONFIG8, CONFIG9
- sheet Transceiver pair1 ports: added CONFIG_CLK, CONFIG_CLR_N, CONFIG_DATA_IN, CONFIG_DATA_OUT, CONFIG_OE_N, CONFIG_UPDATE, FPGA_MUX_IN_A, FPGA_MUX_IN_B, FPGA_MUX_OUT_A, FPGA_MUX_OUT_B, LED_GRN, LED_YLW; removed 1BIAS+, 1BIAS-, 2BIAS+, 2BIAS-, CONFIG1, CONFIG10, CONFIG2, CONFIG3, CONFIG4, CONFIG5, CONFIG6, CONFIG7, CONFIG8, CONFIG9

Commit message: add current limit and sense parts, add possible endat solution
Other:
- sheet Port Power ports: added FAULT_N_VH_BANK_1, FAULT_N_VH_BANK_2, FAULT_N_VL_BANK_1, FAULT_N_VL_BANK_2; removed none
- sheet Transceiver pair ports: added MUX_A, MUX_B; removed FPGA_MUX_IN_A, FPGA_MUX_IN_B, FPGA_MUX_OUT_A, FPGA_MUX_OUT_B
- sheet Transceiver pair1 ports: added MUX_A, MUX_B; removed FPGA_MUX_IN_A, FPGA_MUX_IN_B, FPGA_MUX_OUT_A, FPGA_MUX_OUT_B
- sheet Transceiver pair2 ports: added MUX_A, MUX_B; removed FPGA_MUX_IN_A, FPGA_MUX_IN_B, FPGA_MUX_OUT_A, FPGA_MUX_OUT_B
- sheet Transceiver pair3 ports: added MUX_A, MUX_B; removed FPGA_MUX_IN_A, FPGA_MUX_IN_B, FPGA_MUX_OUT_A, FPGA_MUX_OUT_B
- sheet Transceiver pair4 ports: added MUX_A, MUX_B; removed FPGA_MUX_IN_A, FPGA_MUX_IN_B, FPGA_MUX_OUT_A, FPGA_MUX_OUT_B
- sheet Transceiver pair5 ports: added MUX_A, MUX_B; removed FPGA_MUX_IN_A, FPGA_MUX_IN_B, FPGA_MUX_OUT_A, FPGA_MUX_OUT_B
- sheet Transceiver pair6 ports: added MUX_A, MUX_B; removed FPGA_MUX_IN_A, FPGA_MUX_IN_B, FPGA_MUX_OUT_A, FPGA_MUX_OUT_B
- sheet Transceiver pair7 ports: added MUX_A, MUX_B; removed FPGA_MUX_IN_A, FPGA_MUX_IN_B, FPGA_MUX_OUT_A, FPGA_MUX_OUT_B
