File: KiCad/Serial Module/transceivers.kicad_sch (KiCad schematic)
At the start: 17 parts

Commit message: Serial Module: review fixes, full BOM part numbers, stock footprints
Schematic fixes:
- +24V_PORT tied to +24V; STM32 VBAT tied to VDD
- Pull-ups on CONFIG15-18 and on bias-buffer OE inputs; pull-downs on PC13/PC14
- CONFIG_UPDATE moved from PC15 to PC7; VCXO Vcon biased to 1.65 V
- RJ45 LED anodes moved from 5V_LOGIC to 3.3V
- 74LVC125 units kept within one transceiver-pair instance; fixed pair-1
  annotation (U27/U28 units) that shorted MUX_B to DI_B in the netlist
- 5 V bias buffers changed to TI SN74ACT125PWR (TTL inputs, 4.5-5.5 V)
- Current-limit NMOS changed to AO3400A (Transistor_FET symbol, SOT-23 G/S/D)
- 24 V input TVS changed to TI TVS2700DRVR flat-clamp (27 V standoff,
  35 V max clamp at 40 A) replacing PTVS26VZ1USK (42 V clamp)
- Removed unused port_vsense_muc.kicad_sch

BOM and footprints:
- Every part now has Manufacturer, Part number and LCSC# (verified in stock);
  YAGEO caps/resistors, TI logic where stocked
- 24 V-rail MLCCs now 10 uF 50 V X7R 1210; bulk caps 100 uF 50 V
- TPS274160B footprint corrected to VQFN-28 4x5 mm (RLH); THVD1420 to
  150-mil SOIC-8; all custom footprints replaced with KiCad stock except
  J1 (card connector) and J3 (2x4 RJ45)
- "Part Number" fields normalised to "Part number"

Co-Authored-By: Claude Opus 5.5 <noreply@anthropic.com>
Parts:
- J3: value ~ -> (none); Manufacturer (none) -> HCTL; Part number (none) -> HC-RJ45-059D-2*4-2-04
- R45, R46, R47, R48, R49, R50, R51, R52, R53, R54, R55, R56, R57, R58, R59, R60: LCSC# (none) -> C22548; Manufacturer (none) -> YAGEO; Part number (none) -> RC0603FR-071KL
Connections:
- net +5V_LOGIC renamed +3.3V
