File: KiCad/Serial Module/MCU.kicad_sch (KiCad schematic)
At the start: 34 parts, among them J2 Conn_ARM_SWD_TagConnect_TC2030, U1 STM32F411RETx, U7 74LVC1G126, U8 74LVC1G126, X1 25Mhz

Commit message: Serial Module: review fixes, full BOM part numbers, stock footprints
Schematic fixes:
- +24V_PORT tied to +24V; STM32 VBAT tied to VDD
- Pull-ups on CONFIG15-18 and on bias-buffer OE inputs; pull-downs on PC13/PC14
- CONFIG_UPDATE moved from PC15 to PC7; VCXO Vcon biased to 1.65 V
- RJ45 LED anodes moved from 5V_LOGIC to 3.3V
- 74LVC125 units kept within one transceiver-pair instance; fixed pair-1
  annotation (U27/U28 units) that shorted MUX_B to DI_B in the netlist
- 5 V bias buffers changed to TI SN74ACT125PWR (TTL inputs, 4.5-5.5 V)
- Current-limit NMOS changed to AO3400A (Transistor_FET symbol, SOT-23 G/S/D)
- 24 V input TVS changed to TI TVS2700DRVR flat-clamp (27 V standoff,
  35 V max clamp at 40 A) replacing PTVS26VZ1USK (42 V clamp)
- Removed unused port_vsense_muc.kicad_sch

BOM and footprints:
- Every part now has Manufacturer, Part number and LCSC# (verified in stock);
  YAGEO caps/resistors, TI logic where stocked
- 24 V-rail MLCCs now 10 uF 50 V X7R 1210; bulk caps 100 uF 50 V
- TPS274160B footprint corrected to VQFN-28 4x5 mm (RLH); THVD1420 to
  150-mil SOIC-8; all custom footprints replaced with KiCad stock except
  J1 (card connector) and J3 (2x4 RJ45)
- "Part Number" fields normalised to "Part number"

Co-Authored-By: Claude Opus 5.5 <noreply@anthropic.com>
Parts:
- added R385, R386, R387, R388: 10k, Resistor_SMD:R_0603_1608Metric, symbol Device:R
- C1, C3: LCSC# (none) -> C277476; Manufacturer (none) -> YAGEO; Part number (none) -> CC0603KRX5R7BB475
- C10, C15, C16, C18: LCSC# C105882 -> C14663; Part number CC0402KRX5R9BB104 -> CC0603KRX7R9BB104
- C14: LCSC# C50254 -> C309478; Manufacturer Samsung Electro-Mechanics -> YAGEO; Part number CL31B225KBHNNNE -> CC0603KRX5R8BB225; cost 0.03 -> 0.0352
- C2, C4, C5, C6, C7, C8, C9: LCSC# (none) -> C14663; Manufacturer (none) -> YAGEO; Part number (none) -> CC0603KRX7R9BB104
- D1, D2, D5: LCSC# (none) -> C2286; Manufacturer (none) -> Hubei KENTO Elec; Part number (none) -> KT-0603R
- J2: Part number (none) -> N/A - Tag-Connect TC2030 pads only (no part placed)
- R1, R2, R6, R9: LCSC# (none) -> C22548; Manufacturer (none) -> YAGEO; Part number (none) -> RC0603FR-071KL
- R25, R3, R4, R5: LCSC# (none) -> C98220; Manufacturer (none) -> YAGEO; Part number (none) -> RC0603FR-0710KL
- R7, R8: footprint Resistor_SMD:R_0603_1608Metric -> Resistor_SMD:R_0402_1005Metric
- U1: footprint footprints:LQFP-64_10x10mm_P0.5mm_smaller_pads -> Package_QFP:LQFP-64_10x10mm_P0.5mm; LCSC# (none) -> C94355; Manufacturer (none) -> STMicroelectronics; Part number (none) -> STM32F411RET6
Connections:
- net +3.3V: now also U1.1 (VBAT), R387.1
- net CONFIG_UPDATE: now also U1.38 (PC7); no longer U1.4 (PC15)
- net GND: now also R385.2, R386.2, R388.2
- net RX_PASSTHROUGH_ENABLE: now also R386.1
- net TX_PASSTHROUGH_ENABLE: now also R385.1
- net at C14.2, C16.2, R8.2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: now also R387.2, R388.1
Other:
- moved on the sheet: C14, C15, C16, R8, X1
