File: KiCad/Serial Module/current_limit_mux.kicad_sch (KiCad schematic)
At the start: 28 parts, among them Q1 NMOS, Q2 NMOS, Q3 NMOS, Q4 NMOS, Q5 NMOS, Q6 NMOS, Q7 NMOS, Q8 NMOS, U88 74HC595

Commit message: Serial Module: review fixes, full BOM part numbers, stock footprints
Schematic fixes:
- +24V_PORT tied to +24V; STM32 VBAT tied to VDD
- Pull-ups on CONFIG15-18 and on bias-buffer OE inputs; pull-downs on PC13/PC14
- CONFIG_UPDATE moved from PC15 to PC7; VCXO Vcon biased to 1.65 V
- RJ45 LED anodes moved from 5V_LOGIC to 3.3V
- 74LVC125 units kept within one transceiver-pair instance; fixed pair-1
  annotation (U27/U28 units) that shorted MUX_B to DI_B in the netlist
- 5 V bias buffers changed to TI SN74ACT125PWR (TTL inputs, 4.5-5.5 V)
- Current-limit NMOS changed to AO3400A (Transistor_FET symbol, SOT-23 G/S/D)
- 24 V input TVS changed to TI TVS2700DRVR flat-clamp (27 V standoff,
  35 V max clamp at 40 A) replacing PTVS26VZ1USK (42 V clamp)
- Removed unused port_vsense_muc.kicad_sch

BOM and footprints:
- Every part now has Manufacturer, Part number and LCSC# (verified in stock);
  YAGEO caps/resistors, TI logic where stocked
- 24 V-rail MLCCs now 10 uF 50 V X7R 1210; bulk caps 100 uF 50 V
- TPS274160B footprint corrected to VQFN-28 4x5 mm (RLH); THVD1420 to
  150-mil SOIC-8; all custom footprints replaced with KiCad stock except
  J1 (card connector) and J3 (2x4 RJ45)
- "Part Number" fields normalised to "Part number"

Co-Authored-By: Claude Opus 5.5 <noreply@anthropic.com>
Parts:
- C157: LCSC# (none) -> C14663; Manufacturer (none) -> YAGEO; Part number (none) -> CC0603KRX7R9BB104
- Q1, Q2, Q3, Q4, Q5, Q6, Q7, Q8: value NMOS -> AO3400A; footprint (none) -> Package_TO_SOT_SMD:SOT-23; symbol Simulation_SPICE:NMOS -> Transistor_FET:AO3400A; LCSC# (none) -> C20917; Manufacturer (none) -> Alpha & Omega Semicon; Part number (none) -> AO3400A
- R253, R257, R262, R264: LCSC# (none) -> C131052; Manufacturer (none) -> YAGEO; Part number (none) -> RC0603FR-078K06L
- R254, R266: LCSC# (none) -> C227925; Manufacturer (none) -> YAGEO; Part number (none) -> AC0603FR-074K02L
- R255, R268: LCSC# (none) -> C105576; Manufacturer (none) -> YAGEO; Part number (none) -> RC0603FR-072KL
- R256, R270: LCSC# (none) -> C22548; Manufacturer (none) -> YAGEO; Part number (none) -> RC0603FR-071KL
- R258, R259, R260, R261, R263, R265, R267, R269: LCSC# (none) -> C98220; Manufacturer (none) -> YAGEO; Part number (none) -> RC0603FR-0710KL
- U88: LCSC# C5948 -> C273642; Manufacturer (none) -> TI; Part number (none) -> SN74HC595PWR
Connections:
- net GND: now also Q1.2 (S), Q2.2 (S), Q3.2 (S), Q4.2 (S), Q5.2 (S), Q6.2 (S), Q7.2 (S), Q8.2 (S); no longer Q1.3 (S), Q2.3 (S), Q3.3 (S), Q4.3 (S), Q5.3 (S), Q6.3 (S), Q7.3 (S), Q8.3 (S)
- net at R268.2: now also Q7.3 (D); no longer Q7.1 (D)
- net at R267.1, U88.6 (QG): now also Q7.1 (G); no longer Q7.2 (G)
- net at R269.1, U88.7 (QH): now also Q8.1 (G); no longer Q8.2 (G)
- net at Q4.1 (G): now also R261.1, U88.3 (QD); no longer R256.2
- net at Q2.1 (G): now also R259.1, U88.1 (QB); no longer R254.2
- net at R255.2: now also Q3.3 (D); no longer Q3.1 (D)
- net at R258.1, U88.15 (QA): now also Q1.1 (G); no longer Q1.2 (G)
- net at R260.1, U88.2 (QC): now also Q3.1 (G); no longer Q3.2 (G)
- net at R263.1, U88.4 (QE): now also Q5.1 (G); no longer Q5.2 (G)
- net at R265.1, U88.5 (QF): now also Q6.1 (G); no longer Q6.2 (G)
- net at R253.2: now also Q1.3 (D); no longer Q1.1 (D)
- net at R270.2: now also Q8.3 (D); no longer Q8.1 (D)
- net at R264.2: now also Q5.3 (D); no longer Q5.1 (D)
- net at R266.2: now also Q6.3 (D); no longer Q6.1 (D)
- new net: Q4.3 (D), R256.2
- new net: Q2.3 (D), R254.2
