File: KiCad/Serial Module/transceiver_pair.kicad_sch (KiCad schematic)
At the start: 54 parts, among them U10 74LVC125, U106 74HC595, U11 THVD1420D, U12 THVD1420D, U16 74HC595, U17 74HC595, U28 74LVC125, U51 74HC595, U66 74LVC125, U9 74LVC125, U90 74LVC125, U98 74LVC125

Commit message: Serial Module: review fixes, full BOM part numbers, stock footprints
Schematic fixes:
- +24V_PORT tied to +24V; STM32 VBAT tied to VDD
- Pull-ups on CONFIG15-18 and on bias-buffer OE inputs; pull-downs on PC13/PC14
- CONFIG_UPDATE moved from PC15 to PC7; VCXO Vcon biased to 1.65 V
- RJ45 LED anodes moved from 5V_LOGIC to 3.3V
- 74LVC125 units kept within one transceiver-pair instance; fixed pair-1
  annotation (U27/U28 units) that shorted MUX_B to DI_B in the netlist
- 5 V bias buffers changed to TI SN74ACT125PWR (TTL inputs, 4.5-5.5 V)
- Current-limit NMOS changed to AO3400A (Transistor_FET symbol, SOT-23 G/S/D)
- 24 V input TVS changed to TI TVS2700DRVR flat-clamp (27 V standoff,
  35 V max clamp at 40 A) replacing PTVS26VZ1USK (42 V clamp)
- Removed unused port_vsense_muc.kicad_sch

BOM and footprints:
- Every part now has Manufacturer, Part number and LCSC# (verified in stock);
  YAGEO caps/resistors, TI logic where stocked
- 24 V-rail MLCCs now 10 uF 50 V X7R 1210; bulk caps 100 uF 50 V
- TPS274160B footprint corrected to VQFN-28 4x5 mm (RLH); THVD1420 to
  150-mil SOIC-8; all custom footprints replaced with KiCad stock except
  J1 (card connector) and J3 (2x4 RJ45)
- "Part Number" fields normalised to "Part number"

Co-Authored-By: Claude Opus 5.5 <noreply@anthropic.com>
Parts:
- added R321, R322, R323, R324, R353, R354, R355, R356: 10K, Resistor_SMD:R_0603_1608Metric, symbol Device:R
- added unit 2 of U90
- added unit 3 of U98
- added unit 4 of U98
- added unit 2 of U98
- added unit 5 of U98
- C111, C159, C167, C17, C175, C19, C25, C26, C31, C32, C96: LCSC# (none) -> C14663; Manufacturer (none) -> YAGEO; Part number (none) -> CC0603KRX7R9BB104
- D6, D7: LCSC# (none) -> C172881; Manufacturer (none) -> Littelfuse; Part number (none) -> SM712-02HTG
- R10, R11, R12, R13, R159, R171, R179, R187, R195, R203, R211, R219, R227, R235, R289, R297, R305, R313: LCSC# (none) -> C98220; Manufacturer (none) -> YAGEO; Part number (none) -> RC0603FR-0710KL
- R14, R15, R16, R17: LCSC# (none) -> C114669; Manufacturer (none) -> YAGEO; Part number (none) -> RC0603FR-07470RL
- R18, R19: LCSC# (none) -> C109318; Manufacturer (none) -> YAGEO; Part number (none) -> RC0603FR-0710RL
- R20, R21: LCSC# (none) -> C138066; Manufacturer (none) -> YAGEO; Part number (none) -> RC0402FR-0710RL
- R22, R23: LCSC# (none) -> C227580; Manufacturer (none) -> YAGEO; Part number (none) -> AC0603FR-07137RL
- U10, U9, U90, U98: footprint Package_DFN_QFN:DHVQFN-14-1EP_2.5x3mm_P0.5mm_EP1x1.5mm -> Package_SO:TSSOP-14_4.4x5mm_P0.65mm; LCSC# C54411083 -> C7813; Manufacturer (none) -> TI; Part number (none) -> SN74LVC125APWR
- U106, U16, U17, U51: LCSC# C5948 -> C273642; Manufacturer (none) -> TI; Part number (none) -> SN74HC595PWR
- U11, U12: footprint footprints:SOIC-8_4.9x3.91mm_P1.27mm -> Package_SO:SOIC-8_3.9x4.9mm_P1.27mm; Part Number THVD1420DR -> (none); Part number (none) -> THVD1420DR
- U66: value 74LVC125 -> 74ACT125; footprint Package_DFN_QFN:DHVQFN-14-1EP_2.5x3mm_P0.5mm_EP1x1.5mm -> Package_SO:TSSOP-14_4.4x5mm_P0.65mm; LCSC# (none) -> C52940839; Manufacturer (none) -> TI; Part number (none) -> SN74ACT125PWR
- U90: renamed from U28; footprint Package_DFN_QFN:DHVQFN-14-1EP_2.5x3mm_P0.5mm_EP1x1.5mm -> Package_SO:TSSOP-14_4.4x5mm_P0.65mm; LCSC# C54411083 -> C7813; Manufacturer (none) -> TI; Part number (none) -> SN74LVC125APWR
Connections:
- net +3.3V: now also R321.2, R322.2, R323.2, R324.2, R353.2, R354.2, R355.2, R356.2, U98.14 (VCC); no longer U98.14 (VCC)
- net CONFIG11: now also U90.4; no longer U90.1
- net CONFIG12: now also U90.1; no longer U90.4
- net CONFIG13: now also U90.13; no longer U90.10
- net CONFIG14: now also U90.10; no longer U90.13
- net CONFIG15: now also R321.1
- net CONFIG16: now also R322.1, U98.4; no longer U98.4
- net CONFIG17: now also R323.1, U98.10; no longer U98.10
- net CONFIG18: now also R324.1, U98.13; no longer U98.13
- net DI_A: now also U90.6, U98.6; no longer U90.3, U98.6
- net DI_B: now also U90.11, U98.11, U98.8; no longer U90.8, U98.11, U98.8
- net FPGA_A: now also U90.12, U90.2; no longer U90.5, U90.9
- net FPGA_B: now also U90.9, U90.5; no longer U90.12, U90.2
- net GND: now also U98.7 (GND); no longer U98.7 (GND)
- net MUX_A: now also U90.3, U98.9; no longer U90.6, U98.9
- net MUX_B: now also U90.8, U98.12, U98.5; no longer U90.11, U98.12, U98.5
- net QF: now reaches U51.5 (QF), U66.10
- net QF: now also R355.1
- net QD: now reaches U51.3 (QD), U66.4
- net QD: now also R354.1
- net QH: now reaches U51.7 (QH), U66.13
- net QH: now also R356.1
- net QB: now reaches U51.1 (QB), U66.1
- net QB: now also R353.1
Other:
- moved on the sheet: C140, R159, R171, R179, R187, R195, R203, R211, R219, R227, R235, R289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

Commit message: Serial Module: move 3.3 V 74LVC125 buffers back to 2.5x3 mm DHVQFN-14
The 32 3.3 V buffers return to Nexperia 74LVC125ABQ,115 (LCSC C282343,
DHVQFN-14 2.5x3 mm) from TI SN74LVC125APWR (TSSOP-14) to recover board
area. TI's same-size SN74LVC125ABQAR has only ~96 units at LCSC.

Co-Authored-By: Claude Opus 5.5 <noreply@anthropic.com>
Parts:
- U10, U9, U90, U98: footprint Package_SO:TSSOP-14_4.4x5mm_P0.65mm -> Package_DFN_QFN:DHVQFN-14-1EP_2.5x3mm_P0.5mm_EP1x1.5mm; LCSC# C7813 -> C282343; Manufacturer TI -> Nexperia; Part number SN74LVC125APWR -> 74LVC125ABQ,115
